File: cores/simson/sch/sound.kicad_sch (KiCad schematic)
At the start: 18 parts, among them CN2 Conn_02x16_Row_Letter_Last

Commit message: wip obj simson
Parts:
- renumbered C7 to C?, C6 to C?, C8 to C?, CN2 to CN?, D14 to D?, D2 to D?, D13 to D?, D6 to D?, E16 to E?, E4 to E?, F1 to F?, F3 to F?, F5 to F?, F6 to F?, F2 to F?, R17 to R?, RN14 to RN?, RN15 to RN?
Connections:
- net R_A0 renamed R_MAIN_A0
- net SND_A0 renamed SND_MAIN_A0
