File: cores/simson/sch/colmix.kicad_sch (KiCad schematic)
At the start: 8 parts, among them J10 74LS157, J11 74LS157, J9 74LS157, K13 053251

Commit message: wip obj simson
Parts:
- renumbered F18 to F?, H9 to G8, H10 to G9, J11 to H7, J9 to H8, J10 to H9, H11 to H?, K13 to K?
Connections:
- net MAIN_A0 renamed MAIN_MAIN_A0
Other:
- sheet rgb ports: added MAIN_DB[7..0]; removed MAIN_D[15..0]
Changed lines of the file:
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@@
     (effects (font (size 1.27 1.27)) (justify left bottom))
   )
-  (label "MAIN_A0" (at 158.75 82.55 270) (fields_autoplaced)
+  (label "MAIN_MAIN_A0" (at 158.75 82.55 270) (fields_autoplaced)
     (effects (font (size 1.27 1.27)) (justify right bottom))
   )
@@
     (effects (font (size 1.27 1.27)) (justify right))
   )
-  (hierarchical_label "MAIN_D[15..0]" (shape bidirectional) (at 231.14 269.24 180) (fields_autoplaced)
+  (hierarchical_label "MAIN_D[7..0]" (shape bidirectional) (at 231.14 269.24 180) (fields_autoplaced)
     (effects (font (size 1.27 1.27)) (justify right))
   )
@@
   (symbol (lib_id "konami:053251") (at 146.05 140.97 0) (unit 1)
     (in_bom yes) (on_board yes) (dnp no)
-    (property "Reference" "K13" (at 146.05 133.35 0)
+    (property "Reference" "K?" (at 146.05 133.35 0)
       (effects (font (size 1.27 1.27)))
     )
@@
       (project "tsimpsons"
         (path "/b2532043-1bc6-481f-b85e-02a5b9b5cc00/b7286211-d54d-4da5-b787-d67d10f33c0b"
-          (reference "K13") (unit 1)
+          (reference "K?") (unit 1)
         )
       )
@@
   (symbol (lib_id "jt74:74LS04") (at 191.77 90.17 180) (unit 5)
     (in_bom yes) (on_board yes) (dnp no)
-    (property "Reference" "H11" (at 191.77 91.44 0)
+    (property "Reference" "H?" (at 191.77 91.44 0)
       (effects (font (size 1.27 1.27)))
     )
@@
       (project "tsimpsons"
         (path "/b2532043-1bc6-481f-b85e-02a5b9b5cc00/b7286211-d54d-4da5-b787-d67d10f33c0b"
-          (reference "H11") (unit 5)
+          (reference "H?") (unit 5)
         )
       )
@@
   (symbol (lib_id "power:VSS") (at 187.96 191.77 180) (unit 1)
     (in_bom yes) (on_board yes) (dnp no)
-    (property "Reference" "#PWR0111" (at 187.96 187.96 0)
+    (property "Reference" "#PWR?" (at 187.96 187.96 0)
       (effects (font (size 1.27 1.27)) hide)
     )
@@
       (project "tsimpsons"
         (path "/b2532043-1bc6-481f-b85e-02a5b9b5cc00/b7286211-d54d-4da5-b787-d67d10f33c0b"
-          (reference "#PWR0111") (unit 1)
+          (reference "#PWR?") (unit 1)
         )
       )
@@
   (symbol (lib_id "jt74:74LS157") (at 273.05 132.08 0) (unit 1)
     (in_bom yes) (on_board yes) (dnp no)
-    (property "Reference" "J10" (at 278.13 115.57 0)
+    (property "Reference" "H9" (at 278.13 115.57 0)
       (effects (font (size 1.27 1.27)))
     )
@@
       (project "tsimpsons"
         (path "/b2532043-1bc6-481f-b85e-02a5b9b5cc00/b7286211-d54d-4da5-b787-d67d10f33c0b"
-          (reference "J10") (unit 1)
+          (reference "H9") (unit 1)
         )
       )
@@
   (symbol (lib_id "jt74:74LS157") (at 273.05 168.91 0) (unit 1)
     (in_bom yes) (on_board yes) (dnp no)
-    (property "Reference" "J9" (at 278.13 152.4 0)
+    (property "Reference" "H8" (at 278.13 152.4 0)
       (effects (font (size 1.27 1.27)))
     )
@@
       (project "tsimpsons"
         (path "/b2532043-1bc6-481f-b85e-02a5b9b5cc00/b7286211-d54d-4da5-b787-d67d10f33c0b"
-          (reference "J9") (unit 1)
+          (reference "H8") (unit 1)
         )
       )
@@
   (symbol (lib_id "jt74:74LS32") (at 214.63 157.48 0) (unit 3)
     (in_bom yes) (on_board yes) (dnp no)
-    (property "Reference" "F18" (at 214.63 156.21 0)
+    (property "Reference" "F?" (at 214.63 156.21 0)
       (effects (font (size 1.27 1.27)))
     )
@@
       (project "tsimpsons"
         (path "/b2532043-1bc6-481f-b85e-02a5b9b5cc00/b7286211-d54d-4da5-b787-d67d10f33c0b"
-          (reference "F18") (unit 3)
+          (reference "F?") (unit 3)
         )
       )
@@
   (symbol (lib_id "arcade:HM6116P-3") (at 328.93 154.94 0) (unit 1)
     (in_bom yes) (on_board yes) (dnp no)
-    (property "Reference" "H9" (at 328.93 153.67 0)
+    (property "Reference" "G8" (at 328.93 153.67 0)
       (effects (font (size 1.27 1.27)))
     )
@@
       (project "tsimpsons"
         (path "/b2532043-1bc6-481f-b85e-02a5b9b5cc00/b7286211-d54d-4da5-b787-d67d10f33c0b"
-          (reference "H9") (unit 1)
+          (reference "G8") (unit 1)
         )
       )
@@
   (symbol (lib_id "arcade:HM6116P-3") (at 328.93 104.14 0) (unit 1)
     (in_bom yes) (on_board yes) (dnp no)
-    (property "Reference" "H10" (at 328.93 102.87 0)
+    (property "Reference" "G9" (at 328.93 102.87 0)
       (effects (font (size 1.27 1.27)))
     )
@@
       (project "tsimpsons"
         (path "/b2532043-1bc6-481f-b85e-02a5b9b5cc00/b7286211-d54d-4da5-b787-d67d10f33c0b"
-          (reference "H10") (unit 1)
+          (reference "G9") (unit 1)
         )
       )
@@
   (symbol (lib_id "power:VCC") (at 100.33 95.25 0) (unit 1)
     (in_bom yes) (on_board yes) (dnp no)
-    (property "Reference" "#PWR0110" (at 100.33 99.06 0)
+    (property "Reference" "#PWR?" (at 100.33 99.06 0)
       (effects (font (size 1.27 1.27)) hide)
     )
@@
       (project "tsimpsons"
         (path "/b2532043-1bc6-481f-b85e-02a5b9b5cc00/b7286211-d54d-4da5-b787-d67d10f33c0b"
-          (reference "#PWR0110") (unit 1)
+          (reference "#PWR?") (unit 1)
         )
       )
@@
   (symbol (lib_id "jt74:74LS157") (at 273.05 95.25 0) (unit 1)
     (in_bom yes) (on_board yes) (dnp no)
-    (property "Reference" "J11" (at 278.13 78.74 0)
+    (property "Reference" "H7" (at 278.13 78.74 0)
       (effects (font (size 1.27 1.27)))
     )
@@
       (project "tsimpsons"
         (path "/b2532043-1bc6-481f-b85e-02a5b9b5cc00/b7286211-d54d-4da5-b787-d67d10f33c0b"
-          (reference "J11") (unit 1)
+          (reference "H7") (unit 1)
         )
       )
@@
       (effects (font (size 1.27 1.27)) (justify left))
     )
-    (pin "MAIN_D[15..0]" bidirectional (at 238.76 269.24 180)
-      (effects (font (size 1.27 1.27)) (justify left))
-    )
     (pin "~{VBLANK}" input (at 238.76 259.08 180)
       (effects (font (size 1.27 1.27)) (justify left))
@@
       (effects (font (size 1.27 1.27)) (justify left))
     )
+    (pin "MAIN_DB[7..0]" bidirectional (at 238.76 269.24 180)
+      (effects (font (size 1.27 1.27)) (justify left))
+    )

Commit message: wip obj scr simpson
Connections:
- net CRAM~{CS}: no longer H8.14 (I0d)
- new net UK~{RD}: H8.14 (I0d)
Changed lines of the file:
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@@
     (stroke (width 0) (type default))
   )
-  (wire (pts (xy 248.92 163.83) (xy 260.35 163.83))
+  (wire (pts (xy 256.54 163.83) (xy 260.35 163.83))
     (stroke (width 0) (type default))
   )
@@
     (effects (font (size 1.27 1.27)) (justify left bottom))
   )
-  (label "CRAM~{CS}" (at 248.92 163.83 0) (fields_autoplaced)
-    (effects (font (size 1.27 1.27)) (justify left bottom))
-  )
   (label "FCOL0" (at 138.43 204.47 90) (fields_autoplaced)
     (effects (font (size 1.27 1.27)) (justify left bottom))
@@
     (effects (font (size 1.27 1.27)) (justify right bottom))
   )
+  (hierarchical_label "UK~{RD}" (shape input) (at 256.54 163.83 180) (fields_autoplaced)
+    (effects (font (size 1.27 1.27)) (justify right))
+  )
   (hierarchical_label "CRAM~{CS}" (shape input) (at 231.14 251.46 180) (fields_autoplaced)

Commit message: wip scroll simson
Parts:
- removed H?: 74LS04, symbol jt74:74LS04
- gave numbers to parts that had none: 2
Connections:
- net APAL3 is gone; now on net VSS: J10.20 (CI07)
- net APAL4 is gone; now on net VSS: J10.21 (CI08)
- net BPAL3 is gone; now on net VSS: J10.55 (CI27)
- net BPAL4 is gone; now on net VSS: J10.56 (CI28)
- net FPAL3 is gone; now on net VSS: J10.64 (CI37)
- net UK~{RD} is gone; now on net M~{RD}: H8.14 (I0d)
- net ACOL0: now also J10.57 (CI30); no longer J10.4 (CI00)
- net ACOL1: now also J10.58 (CI31); no longer J10.5 (CI01)
- net ACOL2: now also J10.59 (CI32); no longer J10.6 (CI02)
- net ACOL3: now also J10.60 (CI33); no longer J10.7 (CI03)
- net APAL0: now also J10.61 (CI34); no longer J10.8 (CI04)
- net APAL1: now also J10.62 (CI35); no longer J10.9 (CI05)
- net APAL2: now also J10.63 (CI36); no longer J10.10 (CI06)
- net BCOL0: now also J10.66 (CI40); no longer J10.47 (CI20)
- net BCOL1: now also J10.67 (CI41); no longer J10.48 (CI21)
- net BCOL2: now also J10.68 (CI42); no longer J10.49 (CI22)
- net BCOL3: now also J10.69 (CI43); no longer J10.50 (CI23)
- net BPAL0: now also J10.70 (CI44); no longer J10.51 (CI24)
- net BPAL1: now also J10.71 (CI45); no longer J10.52 (CI25)
- net BPAL2: now also J10.72 (CI46); no longer J10.54 (CI26)
- net FCOL0: now also J10.47 (CI20); no longer J10.57 (CI30)
- net FCOL1: now also J10.48 (CI21); no longer J10.58 (CI31)
- net FCOL2: now also J10.49 (CI22); no longer J10.59 (CI32)
- net FCOL3: now also J10.50 (CI23); no longer J10.60 (CI33)
- net FPAL0: now also J10.51 (CI24); no longer J10.61 (CI34)
- net FPAL1: now also J10.52 (CI25); no longer J10.62 (CI35)
- net FPAL2: now also J10.54 (CI26); no longer J10.63 (CI36)
- net OBJCLK6: now also J10.41 (CLK)
- net VCC: no longer J10.66 (CI40)
- net VSS: now also J10.10 (CI06), J10.4 (CI00), J10.5 (CI01), J10.6 (CI02), J10.7 (CI03), J10.8 (CI04), J10.9 (CI05); no longer J10.67 (CI41), J10.68 (CI42), J10.69 (CI43), J10.70 (CI44), J10.71 (CI45), J10.72 (CI46)
- net MAIN_D0 renamed MAIN_DB0
- net MAIN_D1 renamed MAIN_DB1
- net MAIN_D2 renamed MAIN_DB2
- net MAIN_D3 renamed MAIN_DB3
- net MAIN_D4 renamed MAIN_DB4
- net MAIN_D5 renamed MAIN_DB5
- net MAIN_MAIN_A0 renamed MAIN_A0
- net OCOL4 renamed PAL0
- net OCOL5 renamed PAL1
- net OCOL6 renamed PAL2
- net OCOL7 renamed PAL3
- net OCOL8 renamed PAL4
Other:
- note added: "6M"
- note removed: "FIX"
- note removed: "SCRA"
- note removed: "SCRB"

Commit message: sch obj scr colmix the simpsons
Parts:
- added F10, F9: 74LS32, symbol jt74:74LS32
- added U2: 74LS04, symbol jt74:74LS04
Connections:
- net MAIN_A11 is gone; now on net MAIN_A10: H8.11 (I0c)
- net MAIN_A0: now also H7.2 (I0a), F10.2, U2.11
- net MAIN_A1: now also H7.5 (I0b); no longer H7.2 (I0a)
- net MAIN_A10: no longer H8.5 (I0b)
- net MAIN_A2: now also H7.11 (I0c); no longer H7.5 (I0b)
- net MAIN_A3: now also H7.14 (I0d); no longer H7.11 (I0c)
- net MAIN_A4: now also H9.2 (I0a); no longer H7.14 (I0d)
- net MAIN_A5: now also H9.5 (I0b); no longer H9.2 (I0a)
- net MAIN_A6: now also H9.11 (I0c); no longer H9.5 (I0b)
- net MAIN_A7: now also H9.14 (I0d); no longer H9.11 (I0c)
- net MAIN_A8: now also H8.2 (I0a); no longer H9.14 (I0d)
- net MAIN_A9: now also H8.5 (I0b); no longer H8.2 (I0a)
- net MCO~{WR}H: no longer names the net of G8.21 (~{WR})
- net MCO~{WR}H: now also F9.6
- net MCO~{WR}L: no longer names the net of G9.21 (~{WR})
- net MCO~{WR}L: now also F9.11
- new net: F10.3, F9.5
- new net: F9.12, F9.8
- new net: F9.9, U2.10
- new net COLO~{CS}: F10.1, F9.10
- new net DS: F9.13, F9.4
Other:
- moved on the sheet: F12C, G8, G9, H7, H8, H9, J10
