File: cores/twin16/sch/fround/GFX-Tiles.kicad_sch (KiCad schematic)
At the start: 31 parts, among them U108 74LS157, U110 74LS257, U112 74LS157, U114 74LS257, U116 74LS157, U132 74LS374, U134 74LS374, U136 MX23C4100, U138 MX23C4100, U140 74LS157, U188 74LS32, U189 74LS32, U195 74LS32, U211 74LS08, U216 74LS04, U218 74LS32, U31 74LS245, U33 74LS245, U34 007779, U36 6264SL, U38 6264SL, U45 007781, U52 74LS174, U54 74LS174, U79 74LS374, U81 74LS374, U83 74LS257, U87 74LS374, U91 74LS257, U92 74LS374, U93 74LS157

Commit message: sch updates from public branch
Changed lines of the file:
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@@
   )
   (symbol (lib_id "power:VCC") (at 273.05 104.14 0) (unit 1)
-    (in_bom yes) (on_board yes) (dnp no) (fields_autoplaced)
+    (in_bom yes) (on_board yes) (dnp no)
     (property "Reference" "#PWR0188" (at 273.05 107.95 0)
       (effects (font (size 1.27 1.27)) hide)
     )
-    (property "Value" "VCC" (at 273.05 99.06 0)
+    (property "Value" "VCC" (at 273.05 100.33 0)
       (effects (font (size 1.27 1.27)))
     )
@@
   )
   (symbol (lib_id "power:GND") (at 271.78 170.18 0) (unit 1)
-    (in_bom yes) (on_board yes) (dnp no) (fields_autoplaced)
+    (in_bom yes) (on_board yes) (dnp no)
     (property "Reference" "#PWR0186" (at 271.78 176.53 0)
       (effects (font (size 1.27 1.27)) hide)
