File: cores/asterix/sch/asterix.kicad_sch (KiCad schematic)
At the start: 2 parts

Commit message: wip main sch asterix
Parts:
- added D17: 74LS157, symbol jt74:74LS157
Connections:
- new net RAM~{OE}: D17.1 (SELECT_~{A}-B)
Other:
- sheet objects ports: added M~{RD}, ~{SYSRES}; removed ~{RESET}
Changed lines of the file:
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@@
+    (stroke (width 0) (type default))
+  )
+  (wire (pts (xy 96.52 273.05) (xy 80.01 273.05))
     (stroke (width 0) (type default))
   )
@@
   )
   (wire (pts (xy 92.71 81.28) (xy 92.71 83.82))
+    (stroke (width 0) (type default))
+  )
+  (wire (pts (xy 311.15 72.39) (xy 327.66 72.39))
     (stroke (width 0) (type default))
   )
@@
     (effects (font (size 1.27 1.27)) (justify left bottom))
   )
-  (label "~{RESET}" (at 311.15 57.15 0) (fields_autoplaced)
+  (label "~{SYSRES}" (at 311.15 57.15 0) (fields_autoplaced)
     (effects (font (size 1.27 1.27)) (justify left bottom))
   )
@@
     (effects (font (size 1.27 1.27)) (justify right bottom))
   )
+  (label "M~{RD}" (at 311.15 72.39 0) (fields_autoplaced)
+    (effects (font (size 1.27 1.27)) (justify left bottom))
+  )
   (label "1P_UP" (at 39.37 123.19 0) (fields_autoplaced)
     (effects (font (size 1.27 1.27)) (justify left bottom))
@@
   )
   (hierarchical_label "MAIN_D'[11..0]" (shape output) (at 41.91 203.2 180) (fields_autoplaced)
+    (effects (font (size 1.27 1.27)) (justify right))
+  )
+  (hierarchical_label "RAM~{OE}" (shape input) (at 80.01 273.05 180) (fields_autoplaced)
     (effects (font (size 1.27 1.27)) (justify right))
   )
@@
     )
   )
+  (symbol (lib_id "jt74:74LS157") (at 109.22 261.62 0) (unit 1)
+    (in_bom yes) (on_board yes) (dnp no)
+    (property "Reference" "D17" (at 114.3 245.11 0)
+      (effects (font (size 1.27 1.27)))
+    )
+    (property "Value" "74LS157" (at 109.22 278.13 0)
+      (effects (font (size 1.27 1.27)))
+    )
+    (property "Footprint" "" (at 109.22 261.62 0)
+      (effects (font (size 1.27 1.27)) hide)
+    )
+    (property "Datasheet" "https://www.alldatasheet.com/datasheet-pdf/pdf/27402/TI/74LS157.html" (at 109.22 280.67 0)
+      (effects (font (size 1.27 1.27)) hide)
+    )
+    (pin "1")
+    (pin "10")
+    (pin "11")
+    (pin "12")
+    (pin "13")
+    (pin "14")
+    (pin "15")
+    (pin "2")
+    (pin "3")
+    (pin "4")
+    (pin "5")
+    (pin "6")
+    (pin "7")
+    (pin "9")
+    (instances
+      (project "asterix"
+        (path "/0011ec10-82c4-4039-b424-337480f568e8/7d4ab3ba-37fa-4111-bbdb-c99f1a708a52"
+          (reference "D17") (unit 1)
+        )
+        (path "/0011ec10-82c4-4039-b424-337480f568e8"
+          (reference "D17") (unit 1)
+        )
+      )
+    )
+  )
   (symbol (lib_id "jt74:74LS153") (at 78.74 223.52 0) (unit 1)
     (in_bom yes) (on_board yes) (dnp no)
@@
     )
   )
-  (sheet (at 327.66 36.83) (size 38.1 35.56) (fields_autoplaced)
+  (sheet (at 327.66 36.83) (size 38.1 39.37) (fields_autoplaced)
     (stroke (width 0.1524) (type solid))
     (fill (color 0 0 0 0.0000))
@@
       (effects (font (size 1.27 1.27)) (justify left bottom))
     )
-    (property "Sheetfile" "objects.kicad_sch" (at 327.66 72.9746 0)
+    (property "Sheetfile" "objects.kicad_sch" (at 327.66 76.7846 0)
       (effects (font (size 1.27 1.27)) (justify left top))
     )
@@
       (effects (font (size 1.27 1.27)) (justify left))
     )
-    (pin "~{RESET}" input (at 327.66 57.15 180)
-      (effects (font (size 1.27 1.27)) (justify left))
-    )
     (pin "~{UDS}" input (at 327.66 67.31 180)
       (effects (font (size 1.27 1.27)) (justify left))
@@
       (effects (font (size 1.27 1.27)) (justify right))
     )
+    (pin "~{SYSRES}" input (at 327.66 57.15 180)
+      (effects (font (size 1.27 1.27)) (justify left))
+    )
+    (pin "M~{RD}" input (at 327.66 72.39 180)
+      (effects (font (size 1.27 1.27)) (justify left))
+    )
     (instances

Commit message: main done. wip colmix asterix
Changed lines of the file:
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@@
+    (effects (font (size 1.27 1.27)) (justify left bottom))
+  )
+  (text "OK" (at 260.35 119.38 0)
     (effects (font (size 1.27 1.27)) (justify left bottom))
   )

Commit message: uk konami 054358 done. wip colmix
Changed lines of the file:
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@@
     )
+  )
+  (text "OK" (at 262.89 234.95 0)
+    (effects (font (size 1.27 1.27)) (justify left bottom))
   )
   (text "OK" (at 184.15 109.22 0)

Commit message: colmix done. wip scroll asterix
Connections:
- net RAM~{OE}: no longer names the net of D17.1 (SELECT_~{A}-B)
Other:
- sheet colmix ports: added ACOL[3..0], APAL[2..0], BCOL[3..0], BPAL[2..0], CPG~{CS}, FCOL[3..0], FPAL[2..0], MAIN_A[11..1], MAIN_D[15..0], M~{RD}, OCOL[8..0], PAL~{CS}, PR[14..13], SCRCLK6, ~{WE}H, ~{WE}L; removed BRIT, BRITEN, BRIT[2..0], DFI[7..0], DSA[7..0], DSB[7..0], M6, MAIN_A0, MAIN_A[10..0], MAIN_DB[7..0], M~{DS}, OBJPXL[8..0], PALETTE~{CS}, PAL_BANK, PR13, PR14, R/~{W}, ~{PCU_CS}
Changed lines of the file:
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@@
-    (stroke (width 0) (type default))
-  )
-  (wire (pts (xy 96.52 273.05) (xy 80.01 273.05))
     (stroke (width 0) (type default))
   )
@@
     (effects (font (size 1.27 1.27)) (justify right))
   )
-  (hierarchical_label "RAM~{OE}" (shape input) (at 80.01 273.05 180) (fields_autoplaced)
-    (effects (font (size 1.27 1.27)) (justify right))
-  )
   (symbol (lib_id "arcade:JAMMA_CONN") (at 54.61 78.74 0) (unit 1)
     (in_bom yes) (on_board yes) (dnp no)
@@
     )
   )
-  (sheet (at 327.66 166.37) (size 38.1 53.34) (fields_autoplaced)
+  (sheet (at 327.66 166.37) (size 38.1 62.23) (fields_autoplaced)
     (stroke (width 0.1524) (type solid))
     (fill (color 0 0 0 0.0000))
@@
       (effects (font (size 1.27 1.27)) (justify left bottom))
     )
-    (property "Sheetfile" "colmix.kicad_sch" (at 327.66 220.2946 0)
+    (property "Sheetfile" "colmix.kicad_sch" (at 327.66 229.1846 0)
       (effects (font (size 1.27 1.27)) (justify left top))
     )
-    (pin "OBJPXL[8..0]" input (at 327.66 168.91 180)
-      (effects (font (size 1.27 1.27)) (justify left))
-    )
-    (pin "SDI0" output (at 365.76 171.45 0)
-      (effects (font (size 1.27 1.27)) (justify right))
-    )
-    (pin "M6" input (at 327.66 171.45 180)
-      (effects (font (size 1.27 1.27)) (justify left))
-    )
-    (pin "M~{DS}" input (at 327.66 173.99 180)
-      (effects (font (size 1.27 1.27)) (justify left))
-    )
-    (pin "BRIT" output (at 365.76 168.91 0)
-      (effects (font (size 1.27 1.27)) (justify right))
-    )
-    (pin "PR13" input (at 327.66 186.69 180)
-      (effects (font (size 1.27 1.27)) (justify left))
-    )
-    (pin "PR14" input (at 327.66 189.23 180)
-      (effects (font (size 1.27 1.27)) (justify left))
-    )
-    (pin "R{slash}~{W}" input (at 327.66 191.77 180)
-      (effects (font (size 1.27 1.27)) (justify left))
-    )
-    (pin "MAIN_A0" input (at 327.66 194.31 180)
-      (effects (font (size 1.27 1.27)) (justify left))
-    )
-    (pin "MAIN_A[10..0]" input (at 327.66 199.39 180)
-      (effects (font (size 1.27 1.27)) (justify left))
-    )
-    (pin "PALETTE~{CS}" input (at 327.66 201.93 180)
+    (pin "BLUE" output (at 365.76 176.53 0)
+      (effects (font (size 1.27 1.27)) (justify right))
+    )
+    (pin "RED" output (at 365.76 173.99 0)
+      (effects (font (size 1.27 1.27)) (justify right))
+    )
+    (pin "GREEN" output (at 365.76 179.07 0)
+      (effects (font (size 1.27 1.27)) (justify right))
+    )
+    (pin "SCRCLK6" input (at 327.66 171.45 180)
+      (effects (font (size 1.27 1.27)) (justify left))
+    )
+    (pin "PR[14..13]" input (at 327.66 189.23 180)
+      (effects (font (size 1.27 1.27)) (justify left))
+    )
+    (pin "MAIN_A[11..1]" input (at 327.66 199.39 180)
+      (effects (font (size 1.27 1.27)) (justify left))
+    )
+    (pin "SDI0" input (at 327.66 212.09 180)
+      (effects (font (size 1.27 1.27)) (justify left))
+    )
+    (pin "OCOL[8..0]" input (at 327.66 168.91 180)
+      (effects (font (size 1.27 1.27)) (justify left))
+    )
+    (pin "FCOL[3..0]" input (at 327.66 179.07 180)
+      (effects (font (size 1.27 1.27)) (justify left))
+    )
+    (pin "FPAL[2..0]" input (at 327.66 181.61 180)
+      (effects (font (size 1.27 1.27)) (justify left))
+    )
+    (pin "ACOL[3..0]" input (at 327.66 214.63 180)
+      (effects (font (size 1.27 1.27)) (justify left))
+    )
+    (pin "APAL[2..0]" input (at 327.66 219.71 180)
+      (effects (font (size 1.27 1.27)) (justify left))
+    )
+    (pin "BCOL[3..0]" input (at 327.66 222.25 180)
+      (effects (font (size 1.27 1.27)) (justify left))
+    )
+    (pin "BPAL[2..0]" input (at 327.66 217.17 180)
+      (effects (font (size 1.27 1.27)) (justify left))
+    )
+    (pin "CPG~{CS}" input (at 327.66 184.15 180)
+      (effects (font (size 1.27 1.27)) (justify left))
+    )
+    (pin "PAL~{CS}" input (at 327.66 201.93 180)
+      (effects (font (size 1.27 1.27)) (justify left))
+    )
+    (pin "~{WE}L" input (at 327.66 191.77 180)
+      (effects (font (size 1.27 1.27)) (justify left))
+    )
+    (pin "~{WE}H" input (at 327.66 194.31 180)
+      (effects (font (size 1.27 1.27)) (justify left))
+    )
+    (pin "~{SYSRES}" input (at 327.66 196.85 180)
       (effects (font (size 1.27 1.27)) (justify left))
     )
@@
       (effects (font (size 1.27 1.27)) (justify left))
     )
-    (pin "~{SYSRES}" input (at 327.66 207.01 180)
-      (effects (font (size 1.27 1.27)) (justify left))
-    )
-    (pin "MAIN_DB[7..0]" input (at 327.66 209.55 180)
-      (effects (font (size 1.27 1.27)) (justify left))
-    )
-    (pin "BRITEN" input (at 327.66 212.09 180)
+    (pin "MAIN_D[15..0]" bidirectional (at 327.66 209.55 180)
+      (effects (font (size 1.27 1.27)) (justify left))
+    )
+    (pin "M~{RD}" input (at 327.66 173.99 180)
       (effects (font (size 1.27 1.27)) (justify left))
     )
@@
       (effects (font (size 1.27 1.27)) (justify left))
     )
-    (pin "BLUE" output (at 365.76 176.53 0)
-      (effects (font (size 1.27 1.27)) (justify right))
-    )
-    (pin "RED" output (at 365.76 173.99 0)
-      (effects (font (size 1.27 1.27)) (justify right))
-    )
-    (pin "GREEN" output (at 365.76 179.07 0)
-      (effects (font (size 1.27 1.27)) (justify right))
-    )
-    (pin "DFI[7..0]" input (at 327.66 179.07 180)
-      (effects (font (size 1.27 1.27)) (justify left))
-    )
-    (pin "DSB[7..0]" input (at 327.66 181.61 180)
-      (effects (font (size 1.27 1.27)) (justify left))
-    )
-    (pin "DSA[7..0]" input (at 327.66 214.63 180)
-      (effects (font (size 1.27 1.27)) (justify left))
-    )
-    (pin "PAL_BANK" input (at 327.66 196.85 180)
-      (effects (font (size 1.27 1.27)) (justify left))
-    )
-    (pin "BRIT[2..0]" input (at 327.66 217.17 180)
-      (effects (font (size 1.27 1.27)) (justify left))
-    )
-    (pin "~{PCU_CS}" input (at 327.66 184.15 180)
-      (effects (font (size 1.27 1.27)) (justify left))
-    )

Commit message: wip scr. wip custom chips konami 054156 57
Parts:
- removed D17: 74LS157, symbol jt74:74LS157
Other:
- sheet main2obj renamed main2scr
- sheet main2scr: file main2obj.kicad_sch -> main2scr.kicad_sch
