File: cores/exed/sch/ram_rom.kicad_sch (KiCad schematic)
At the start: 6 parts, among them K10 74LS138, K9 74LS08, M10 27128, M11 27128, M8 TC5565, M9 27128

Commit message: logics_gates_wip
Other:
- company: (none) -> JOTEGO
- title: (none) -> Exed Exes board B
Changed lines of the file:
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@@
 (kicad_sch (version 20211123) (generator eeschema)
   (paper "A4")
+  (title_block
+    (title "Exed Exes board B")
+    (date "2021")
+    (rev "José Tejada G")
+    (company "JOTEGO")
+    (comment 1 "https://patreon.com/topapate")
+    (comment 2 "Extracted by Jose Tejada, 2021")
+    (comment 3 "supplemented by E.Triana")
+  )
   (junction (at 146.05 189.23) (diameter 0) (color 0 0 0 0)
   )

Commit message: video_wip
Parts:
- renumbered K10 to 10K, M10 to 10M, M11 to 11M, M8 to 8M, K9 to 9K, M9 to 9M
Changed lines of the file:
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@@
   (symbol (lib_id "Memory_EPROM:27128") (at 156.21 46.99 0) (unit 1)
     (in_bom yes) (on_board yes)
-    (property "Reference" "M9" (id 0) (at 161.29 20.32 0))
+    (property "Reference" "9M" (id 0) (at 161.29 20.32 0))
     (property "Value" "27128" (id 1) (at 154.94 45.72 0))
     (property "Footprint" "Package_DIP:DIP-28_W15.24mm" (id 2) (at 156.21 46.99 0)
@@
   (symbol (lib_id "Memory_EPROM:27128") (at 156.21 166.37 0) (unit 1)
     (in_bom yes) (on_board yes)
-    (property "Reference" "M11" (id 0) (at 161.29 139.7 0))
+    (property "Reference" "11M" (id 0) (at 161.29 139.7 0))
     (property "Value" "27128" (id 1) (at 156.21 165.1 0))
     (property "Footprint" "Package_DIP:DIP-28_W15.24mm" (id 2) (at 156.21 166.37 0)
@@
   (symbol (lib_id "Memory_EPROM:27128") (at 156.21 106.68 0) (unit 1)
     (in_bom yes) (on_board yes)
-    (property "Reference" "M10" (id 0) (at 161.29 80.01 0))
+    (property "Reference" "10M" (id 0) (at 161.29 80.01 0))
     (property "Value" "27128" (id 1) (at 156.21 105.41 0))
     (property "Footprint" "Package_DIP:DIP-28_W15.24mm" (id 2) (at 156.21 106.68 0)
@@
   (symbol (lib_name "74LS08_3") (lib_id "74xx:74LS08") (at 81.28 114.3 0) (mirror x) (unit 3)
     (in_bom yes) (on_board yes)
-    (property "Reference" "K9" (id 0) (at 81.28 113.03 0))
+    (property "Reference" "9K" (id 0) (at 81.28 113.03 0))
     (property "Value" "74LS08" (id 1) (at 81.28 115.57 0))
     (property "Footprint" "" (id 2) (at 81.28 114.3 0)
@@
   (symbol (lib_name "74LS08_2") (lib_id "74xx:74LS08") (at 113.03 45.72 180) (unit 4)
     (in_bom yes) (on_board yes)
-    (property "Reference" "K9" (id 0) (at 113.03 44.45 0))
+    (property "Reference" "9K" (id 0) (at 113.03 44.45 0))
     (property "Value" "74LS08" (id 1) (at 113.03 46.99 0))
     (property "Footprint" "" (id 2) (at 113.03 45.72 0)
@@
   (symbol (lib_id "toshiba:TC5565") (at 80.01 53.34 0) (unit 1)
     (in_bom yes) (on_board yes)
-    (property "Reference" "M8" (id 0) (at 87.63 33.02 0))
+    (property "Reference" "8M" (id 0) (at 87.63 33.02 0))
     (property "Value" "TC5565" (id 1) (at 80.01 69.85 0))
     (property "Footprint" "" (id 2) (at 82.55 63.5 0)
@@
   (symbol (lib_id "74xx:74LS08") (at 81.28 99.06 0) (unit 1)
     (in_bom yes) (on_board yes)
-    (property "Reference" "K9" (id 0) (at 81.28 97.79 0))
+    (property "Reference" "9K" (id 0) (at 81.28 97.79 0))
     (property "Value" "74LS08" (id 1) (at 81.28 100.33 0))
     (property "Footprint" "" (id 2) (at 81.28 99.06 0)
@@
   (symbol (lib_id "jt74:74LS138") (at 49.53 109.22 0) (unit 1)
     (in_bom yes) (on_board yes)
-    (property "Reference" "K10" (id 0) (at 55.88 97.79 0))
+    (property "Reference" "10K" (id 0) (at 55.88 97.79 0))
     (property "Value" "74LS138" (id 1) (at 53.34 123.19 0))
     (property "Footprint" "" (id 2) (at 49.53 109.22 0)
@@
   (symbol (lib_name "74LS08_4") (lib_id "74xx:74LS08") (at 81.28 106.68 0) (mirror x) (unit 2)
     (in_bom yes) (on_board yes)
-    (property "Reference" "K9" (id 0) (at 81.28 105.41 0))
+    (property "Reference" "9K" (id 0) (at 81.28 105.41 0))
     (property "Value" "74LS08" (id 1) (at 81.28 107.95 0))
     (property "Footprint" "" (id 2) (at 81.28 106.68 0)

Commit message: exed_cre_wip
Parts:
- added RAA12, RAA13: R_Network08_US, Resistor_THT:R_Array_SIP9, symbol Device:R_Network08_US
Connections:
- net A0: now also RAA12.9 (R8)
- net A1: now also RAA12.8 (R7)
- net A10: now also RAA13.7 (R6)
- net A11: now also RAA13.5 (R4)
- net A12: now also RAA13.2 (R1)
- net A2: now also RAA12.7 (R6)
- net A3: now also RAA12.6 (R5)
- net A4: now also RAA12.5 (R4)
- net A5: now also RAA12.4 (R3)
- net A6: now also RAA12.3 (R2)
- net A7: now also RAA12.2 (R1)
- net A8: now also RAA13.3 (R2)
- net A9: now also RAA13.4 (R3)
- net RDn: now also RAA13.6 (R5)
- net VCC: now also RAA12.1 (common), RAA13.1 (common)
- net WRn: now also RAA13.8 (R7)
- no-connect marks 0 -> 1
Other:
- moved on the sheet: 10K, 9KA, 9KB, 9KC

Commit message: cre_wip
Connections:
- net VCC: now also 10M.1 (VPP), 10M.27 (~{PGM}), 11M.1 (VPP), 11M.27 (~{PGM}), 9M.1 (VPP), 9M.27 (~{PGM})
- net MREQn renamed ~{MREQ}
- net RFSHn renamed ~{RFSH}
- net WRn renamed ~{WR}
Changed lines of the file:
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@@
   (junction (at 144.78 129.54) (diameter 0) (color 0 0 0 0)
   )
+  (junction (at 146.05 182.88) (diameter 0) (color 0 0 0 0)
+  )
+  (junction (at 146.05 63.5) (diameter 0) (color 0 0 0 0)
+  )
   (junction (at 30.48 81.28) (diameter 0) (color 0 0 0 0)
+  )
+  (junction (at 146.05 123.19) (diameter 0) (color 0 0 0 0)
   )
   (no_connect (at 67.31 86.36))
@@
     (stroke (width 0) (type default) (color 0 0 0 0))
   )
+  (wire (pts (xy 146.05 62.23) (xy 146.05 63.5))
+    (stroke (width 0) (type default) (color 0 0 0 0))
+  )
   (wire (pts (xy 171.45 156.21) (xy 166.37 156.21))
     (stroke (width 0) (type default) (color 0 0 0 0))
@@
     (stroke (width 0) (type default) (color 0 0 0 0))
   )
+  (wire (pts (xy 146.05 181.61) (xy 146.05 182.88))
+    (stroke (width 0) (type default) (color 0 0 0 0))
+  )
   (bus (pts (xy 134.62 52.07) (xy 134.62 49.53))
     (stroke (width 0) (type default) (color 0 0 0 0))
@@
     (stroke (width 0) (type default) (color 0 0 0 0))
   )
+  (wire (pts (xy 137.16 63.5) (xy 146.05 63.5))
+    (stroke (width 0) (type default) (color 0 0 0 0))
+  )
   (wire (pts (xy 62.23 124.46) (xy 72.39 124.46))
     (stroke (width 0) (type default) (color 0 0 0 0))
@@
     (stroke (width 0) (type default) (color 0 0 0 0))
   )
+  (wire (pts (xy 146.05 182.88) (xy 146.05 184.15))
+    (stroke (width 0) (type default) (color 0 0 0 0))
+  )
   (wire (pts (xy 73.66 127) (xy 73.66 124.46))
     (stroke (width 0) (type default) (color 0 0 0 0))
@@
     (stroke (width 0) (type default) (color 0 0 0 0))
   )
+  (wire (pts (xy 137.16 123.19) (xy 146.05 123.19))
+    (stroke (width 0) (type default) (color 0 0 0 0))
+  )
   (wire (pts (xy 33.02 53.34) (xy 67.31 53.34))
     (stroke (width 0) (type default) (color 0 0 0 0))
@@
     (stroke (width 0) (type default) (color 0 0 0 0))
   )
+  (wire (pts (xy 146.05 123.19) (xy 146.05 124.46))
+    (stroke (width 0) (type default) (color 0 0 0 0))
+  )
   (bus (pts (xy 30.48 35.56) (xy 30.48 38.1))
     (stroke (width 0) (type default) (color 0 0 0 0))
@@
     (stroke (width 0) (type default) (color 0 0 0 0))
   )
+  (wire (pts (xy 146.05 121.92) (xy 146.05 123.19))
+    (stroke (width 0) (type default) (color 0 0 0 0))
+  )
   (wire (pts (xy 144.78 129.54) (xy 144.78 134.62))
     (stroke (width 0) (type default) (color 0 0 0 0))
@@
     (stroke (width 0) (type default) (color 0 0 0 0))
   )
+  (wire (pts (xy 146.05 63.5) (xy 146.05 64.77))
+    (stroke (width 0) (type default) (color 0 0 0 0))
+  )
   (bus (pts (xy 25.4 26.67) (xy 30.48 26.67))
     (stroke (width 0) (type default) (color 0 0 0 0))
@@
     (stroke (width 0) (type default) (color 0 0 0 0))
   )
+  (bus (pts (xy 120.65 26.67) (xy 134.62 26.67))
+    (stroke (width 0) (type default) (color 0 0 0 0))
+  )
   (bus (pts (xy 173.99 156.21) (xy 173.99 153.67))
     (stroke (width 0) (type default) (color 0 0 0 0))
   )
   (bus (pts (xy 173.99 36.83) (xy 173.99 34.29))
+    (stroke (width 0) (type default) (color 0 0 0 0))
+  )
+  (wire (pts (xy 137.16 182.88) (xy 146.05 182.88))
     (stroke (width 0) (type default) (color 0 0 0 0))
   )
@@
     (effects (font (size 1.27 1.27)) (justify left bottom))
   )
-  (label "WRn" (at 63.5 88.9 0)
+  (label "~{WR}" (at 63.5 88.9 0)
     (effects (font (size 1.2446 1.2446)) (justify left bottom))
   )
@@
     (effects (font (size 1.2446 1.2446)) (justify left bottom))
   )
+  (label "A[13..0]" (at 120.65 26.67 0)
+    (effects (font (size 1.2446 1.2446)) (justify left bottom))
+  )
   (label "A10" (at 140.97 168.91 0)
     (effects (font (size 1.27 1.27)) (justify left bottom))
@@
     (effects (font (size 1.27 1.27)) (justify right bottom))
   )
+  (label "VCC" (at 137.16 182.88 0)
+    (effects (font (size 1.2446 1.2446)) (justify left bottom))
+  )
   (label "ROM~{CE}3" (at 137.16 186.69 0)
     (effects (font (size 1.2446 1.2446)) (justify left bottom))
@@
     (effects (font (size 1.27 1.27)) (justify left bottom))
   )
+  (label "VCC" (at 137.16 123.19 0)
+    (effects (font (size 1.2446 1.2446)) (justify left bottom))
+  )
   (label "A11" (at 140.97 52.07 0)
     (effects (font (size 1.27 1.27)) (justify left bottom))
@@
   (label "A3" (at 34.29 60.96 0)
     (effects (font (size 1.27 1.27)) (justify left bottom))
+  )
+  (label "VCC" (at 137.16 63.5 0)
+    (effects (font (size 1.2446 1.2446)) (justify left bottom))
   )
   (label "D7" (at 171.45 161.29 180)
@@
     )
   )
-  (global_label "WRn" (shape input) (at 99.06 40.64 0) (fields_autoplaced)
+  (global_label "~{WR}" (shape input) (at 99.06 40.64 0) (fields_autoplaced)
     (effects (font (size 1.27 1.27)) (justify left))
     (property "Referencias entre hojas" "${INTERSHEET_REFS}" (id 0) (at 105.2547 40.7194 0)
@@
     )
   )
-  (global_label "RFSHn" (shape input) (at 30.48 134.62 180) (fields_autoplaced)
+  (global_label "~{RFSH}" (shape input) (at 30.48 134.62 180) (fields_autoplaced)
     (effects (font (size 1.27 1.27)) (justify right))
     (property "Referencias entre hojas" "${INTERSHEET_REFS}" (id 0) (at 22.1082 134.6994 0)
@@
     )
   )
-  (global_label "MREQn" (shape input) (at 30.48 137.16 180) (fields_autoplaced)
+  (global_label "~{MREQ}" (shape input) (at 30.48 137.16 180) (fields_autoplaced)
     (effects (font (size 1.27 1.27)) (justify right))
     (property "Referencias entre hojas" "${INTERSHEET_REFS}" (id 0) (at 21.8058 137.2394 0)

Commit message: autoannotation
Parts:
- renumbered 10K to 10K1, 10M to 10M1, 11M to 11M1, 8M to 8M1, 9K to 9K1, 9M to 9M1
Changed lines of the file:
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@@
   (symbol (lib_id "Memory_EPROM:27128") (at 156.21 46.99 0) (unit 1)
     (in_bom yes) (on_board yes)
-    (property "Reference" "9M" (id 0) (at 161.29 20.32 0))
+    (property "Reference" "9M1" (id 0) (at 161.29 20.32 0))
     (property "Value" "27128" (id 1) (at 154.94 45.72 0))
     (property "Footprint" "Package_DIP:DIP-28_W15.24mm" (id 2) (at 156.21 46.99 0)
@@
   (symbol (lib_id "Memory_EPROM:27128") (at 156.21 166.37 0) (unit 1)
     (in_bom yes) (on_board yes)
-    (property "Reference" "11M" (id 0) (at 161.29 139.7 0))
+    (property "Reference" "11M1" (id 0) (at 161.29 139.7 0))
     (property "Value" "27128" (id 1) (at 156.21 165.1 0))
     (property "Footprint" "Package_DIP:DIP-28_W15.24mm" (id 2) (at 156.21 166.37 0)
@@
   (symbol (lib_id "Memory_EPROM:27128") (at 156.21 106.68 0) (unit 1)
     (in_bom yes) (on_board yes)
-    (property "Reference" "10M" (id 0) (at 161.29 80.01 0))
+    (property "Reference" "10M1" (id 0) (at 161.29 80.01 0))
     (property "Value" "27128" (id 1) (at 156.21 105.41 0))
     (property "Footprint" "Package_DIP:DIP-28_W15.24mm" (id 2) (at 156.21 106.68 0)
@@
   (symbol (lib_name "74LS08_3") (lib_id "74xx:74LS08") (at 81.28 134.62 0) (mirror x) (unit 3)
     (in_bom yes) (on_board yes)
-    (property "Reference" "9K" (id 0) (at 81.28 133.35 0))
+    (property "Reference" "9K1" (id 0) (at 81.28 133.35 0))
     (property "Value" "74LS08" (id 1) (at 81.28 135.89 0))
     (property "Footprint" "" (id 2) (at 81.28 134.62 0)
@@
   (symbol (lib_name "74LS08_2") (lib_id "74xx:74LS08") (at 113.03 45.72 180) (unit 4)
     (in_bom yes) (on_board yes)
-    (property "Reference" "9K" (id 0) (at 113.03 44.45 0))
+    (property "Reference" "9K1" (id 0) (at 113.03 44.45 0))
     (property "Value" "74LS08" (id 1) (at 113.03 46.99 0))
     (property "Footprint" "" (id 2) (at 113.03 45.72 0)
@@
   (symbol (lib_id "toshiba:TC5565") (at 80.01 53.34 0) (unit 1)
     (in_bom yes) (on_board yes)
-    (property "Reference" "8M" (id 0) (at 87.63 33.02 0))
+    (property "Reference" "8M1" (id 0) (at 87.63 33.02 0))
     (property "Value" "TC5565" (id 1) (at 80.01 69.85 0))
     (property "Footprint" "" (id 2) (at 82.55 63.5 0)
@@
   (symbol (lib_id "74xx:74LS08") (at 81.28 119.38 0) (unit 1)
     (in_bom yes) (on_board yes)
-    (property "Reference" "9K" (id 0) (at 81.28 118.11 0))
+    (property "Reference" "9K1" (id 0) (at 81.28 118.11 0))
     (property "Value" "74LS08" (id 1) (at 81.28 120.65 0))
     (property "Footprint" "" (id 2) (at 81.28 119.38 0)
@@
   (symbol (lib_id "jt74:74LS138") (at 49.53 129.54 0) (unit 1)
     (in_bom yes) (on_board yes)
-    (property "Reference" "10K" (id 0) (at 55.88 118.11 0))
+    (property "Reference" "10K1" (id 0) (at 55.88 118.11 0))
     (property "Value" "74LS138" (id 1) (at 53.34 143.51 0))
     (property "Footprint" "" (id 2) (at 49.53 129.54 0)
@@
   (symbol (lib_name "74LS08_4") (lib_id "74xx:74LS08") (at 81.28 127 0) (mirror x) (unit 2)
     (in_bom yes) (on_board yes)
-    (property "Reference" "9K" (id 0) (at 81.28 125.73 0))
+    (property "Reference" "9K1" (id 0) (at 81.28 125.73 0))
     (property "Value" "74LS08" (id 1) (at 81.28 128.27 0))
     (property "Footprint" "" (id 2) (at 81.28 127 0)

Commit message: exed_exes_finish
Connections:
- net RDn renamed ~{RD}
Changed lines of the file:
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@@
     (effects (font (size 1.27 1.27)) (justify left bottom))
   )
-  (label "RDn" (at 63.5 93.98 0)
+  (label "~{RD}" (at 63.5 93.98 0)
     (effects (font (size 1.2446 1.2446)) (justify left bottom))
   )
@@
     )
   )
-  (global_label "RDn" (shape input) (at 99.06 48.26 0) (fields_autoplaced)
+  (global_label "~{RD}" (shape input) (at 99.06 48.26 0) (fields_autoplaced)
     (effects (font (size 1.27 1.27)) (justify left))
     (property "Referencias entre hojas" "${INTERSHEET_REFS}" (id 0) (at 105.0732 48.3394 0)
