File: cores/rbike/sch/clocks.kicad_sch (KiCad schematic)
At the start: 2 parts

Commit message: wip gxf
Parts:
- added D2, J20, U?: 74LS04, symbol jt74:74LS04
- added E24, H24, J22: 74LS74, symbol jt74:74LS74
- added F24: 74LS32, symbol jt74:74LS32
- added H21, J21: 74LS08, symbol jt74:74LS08
- added H22: 74LS20, symbol jt74:74LS20
- added L15: 74LS138, symbol jt74:74LS138
Connections:
- net VCC: now also E24.1 (~{R}), E24.4 (~{S}), H24.1 (~{R}), H24.4 (~{S}), U?.14 (VCC)
- net VSS: now also U?.7 (VSS)
- net DCLK1: now reaches H23.13 (Q1)
- net DCLK1: now also D2.1, H24.3 (C)
- new net: E24.3 (C), H24.5 (Q)
- new net: F24.11, H21.2
- new net: E24.2 (D), H22.9
- new net: E24.6 (~{Q}), F24.9
- new net: E24.5 (Q), F24.12
- new net SCU~{CS}: L15.10 (O5)
- new net ~{DCLK2}: D2.2, F24.10, F24.13
- new net ~{HS}: H24.2 (D)
- no-connect marks 1 -> 2
Other:
- note added: "CP JC24,D24,D22,C22"
- moved on the sheet: H23, XTAL2

Commit message: rbike/risle sch updated from public branch
Parts:
- removed unit 2 of F24
- removed L15: 74LS138, symbol jt74:74LS138
- removed U?: 74LS04, symbol jt74:74LS04
- added A4, H6: 74LS04, symbol jt74:74LS04
- added D1, K16: 74LS08, symbol jt74:74LS08
- added D5, K17: 74LS32, symbol jt74:74LS32
- added K18: 74LS74, symbol jt74:74LS74
Connections:
- new net MAINAND1: D1.11
- new net PIN 7BCU: A4.13, D5.12, H6.11

Commit message: fairyland, rbike schematics
Parts:
- removed A4, D2, H6, J20: 74LS04, symbol jt74:74LS04
- removed D1, H21, J21, K16: 74LS08, symbol jt74:74LS08
- removed D5, F24, K17: 74LS32, symbol jt74:74LS32
- removed E24, H24, J22, K18: 74LS74, symbol jt74:74LS74
- removed H22: 74LS20, symbol jt74:74LS20
- removed H23: 74LS163, symbol jt74:74LS163
- removed XTAL2: 28.000MHz, symbol Device:Crystal_GND23_Small
Connections:
- no-connect marks 2 -> 0
Other:
- note removed: "CP JC24,D24,D22,C22"
- company: (none) -> Esperanza Triana
- title: (none) -> Rally Bike

Commit message: sch: changed copyright notice
Other:
- company: Esperanza Triana -> JOTEGO
Changed lines of the file:
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@@
     (date "2023-05-31")
     (rev "José Tejada G.")
-    (company "Esperanza Triana")
+    (company "JOTEGO")
     (comment 1 "www.patreon.com/jotego")
     (comment 2 "JOTEGO")
