File: cores/tfs/sch/fairyland/objects.kicad_sch (KiCad schematic)
At the start: 68 parts, among them IC1 74LS04, IC10 27128, IC11 27128, IC12 74LS194, IC13 74LS194, IC14 74LS74, IC15 74LS08, IC18 74LS161, IC2 74LS107, IC20 74LS139, IC21 74LS298, IC22 74LS194, IC23 74LS194, IC24 74LS74, IC28 74LS161, IC31 74LS298, IC32 27128, IC33 27128, IC34 27128, IC35 27128, IC36 74LS158, IC37 74LS04, IC38 74LS86, IC39 74LS86, IC40 74LS20, IC42 74LS373, IC43 74LS273, IC46 74LS273, IC47 74LS273, IC48 74LS374, IC49 74LS244, IC5 74LS74, IC52 74LS273, IC54 74LS273, IC55 74LS273, IC56 74LS283, IC57 74LS283, IC58 MBM2148, IC59 MBM2148, IC60 74LS244, IC62 74LS298, IC63 74LS374, IC67 MBM2148, IC68 74LS08, IC69 74LS257, IC7 74LS298, IC70 74LS42, IC75 74LS244, IC8 27128, IC82 74LS244, IC83 74LS157, IC84 74LS157, IC85 74LS157, IC86 RAM_2016, IC9 27128, IC90 74LS245, IC92 74LS174, IC93 74LS174, IC96 74LS08

Commit message: wip counters fairyland
Parts:
- added IC45, IC91, IC94: 74LS245, symbol jt74:74LS245
- added IC76, IC77, IC78: MBM2148, symbol arcade:MBM2148
- added IC95: 74LS374, symbol jt74:74LS374
- added ICR1: R_Network08_US, Resistor_THT:R_Array_SIP9, symbol Device:R_Network08_US
Connections:
- net ~{CE0} is gone; now on net ~{OE0}: IC32.20 (~{CE}), IC8.20 (~{CE})
- net ~{CE1} is gone; now on net ~{OE1}: IC33.20 (~{CE}), IC9.20 (~{CE})
- net ~{CE2} is gone; now on net ~{OE2}: IC10.20 (~{CE}), IC34.20 (~{CE})
- net ~{CE3} is gone; now on net ~{OE3}: IC11.20 (~{CE}), IC35.20 (~{CE})
- net D0: no longer IC62.3 (I0a)
- net D1: now also IC7.4 (I0b); no longer IC62.2 (I1a), IC7.2 (I1a)
- net D2: now also IC7.9 (I0c); no longer IC62.4 (I0b), IC7.4 (I0b)
- net D3: now also IC7.7 (I0d); no longer IC62.1 (I1b), IC7.1 (I1b)
- net D4: now also IC21.3 (I0a), IC62.3 (I0a); no longer IC62.9 (I0c), IC7.9 (I0c)
- net D5: now also IC21.4 (I0b), IC62.4 (I0b); no longer IC62.5 (I1c), IC7.5 (I1c)
- net D6: now also IC21.9 (I0c), IC62.9 (I0c); no longer IC62.7 (I0d), IC7.7 (I0d)
- net D7: now also IC21.7 (I0d), IC62.7 (I0d); no longer IC62.6 (I1d), IC7.6 (I1d)
- net VCC: now also IC76.18 (VCC), IC77.18 (VCC), IC78.18 (VCC), ICR1.1 (common)
- net VSS: now also IC76.9 (VSS), IC77.9 (VSS), IC78.9 (VSS)
- net ~{OE0}: no longer IC2.3 (Q), IC2.8 (J), IC48.1 (~{OE}), IC63.1 (~{OE}), IC92.9 (Cp), IC93.9 (Cp)
- net RA0: now reaches IC75.12 (O3a)
- net RA0: now also IC76.5 (A0), IC77.5 (A0), IC78.5 (A0)
- net RA1: now reaches IC75.14 (O2a)
- net RA1: now also IC76.6 (A1), IC77.6 (A1), IC78.6 (A1)
- net RA2: now reaches IC75.16 (O1a)
- net RA2: now also IC76.7 (A2), IC77.7 (A2), IC78.7 (A2)
- net RA3: now reaches IC75.18 (O0a)
- net RA3: now also IC76.4 (A3), IC77.4 (A3), IC78.4 (A3)
- net RA4: now reaches IC75.3 (O3b)
- net RA4: now also IC76.3 (A4), IC77.3 (A4), IC78.3 (A4)
- net RA5: now reaches IC75.5 (O2b)
- net RA5: now also IC76.2 (A5), IC77.2 (A5), IC78.2 (A5)
- net RA6: now reaches IC75.7 (O1b)
- net RA6: now also IC76.1 (A6), IC77.1 (A6), IC78.1 (A6)
- net RA7: now reaches IC75.9 (O0b)
- net RA7: now also IC76.17 (A7), IC77.17 (A7), IC78.17 (A7)
- net CLK': now reaches IC63.11 (Cp)
- net CLK': now also IC2.3 (Q), IC2.8 (J), IC48.11 (Cp), IC92.9 (Cp), IC93.9 (Cp)
- net ~{Mr'}: now reaches IC92.1 (~{Mr})
- net ~{Mr'}: now also IC93.1 (~{Mr})
- net at IC37.12: now also IC63.1 (~{OE})
- net NOT0: now reaches IC37.13
- net NOT0: now also IC82.18 (O0a)
- net at IC93.13 (D4): now also IC91.17 (B1)
- net at IC93.14 (D5): now also IC91.18 (B0)
- net at IC96.11: now also IC37.11, IC48.1 (~{OE}), IC95.17 (D6)
- net MABD7: now reaches IC90.2 (A0)
- net MABD7: now also IC45.9 (A7), IC91.2 (A0), IC94.2 (A0), ICR1.2 (R1)
- net MABD6: now reaches IC90.3 (A1)
- net MABD6: now also IC45.8 (A6), IC91.3 (A1), IC94.3 (A1), ICR1.3 (R2)
- net MABD5: now reaches IC90.4 (A2)
- net MABD5: now also IC45.7 (A5), IC91.4 (A2), IC94.4 (A2), ICR1.4 (R3)
- net MABD4: now reaches IC90.5 (A3)
- net MABD4: now also IC45.6 (A4), IC91.5 (A3), IC94.5 (A3), ICR1.5 (R4)
- net MABD3: now reaches IC90.6 (A4)
- net MABD3: now also IC45.5 (A3), IC91.6 (A4), IC94.6 (A4), ICR1.6 (R5)
- net MABD2: now reaches IC90.7 (A5)
- net MABD2: now also IC45.4 (A2), IC91.7 (A5), IC94.7 (A5), ICR1.7 (R6)
- net MABD1: now reaches IC90.8 (A6)
- net MABD1: now also IC45.3 (A1), IC91.8 (A6), IC94.8 (A6), ICR1.8 (R7)
- net MABD0: now reaches IC90.9 (A7)
- net MABD0: now also IC45.2 (A0), IC91.9 (A7), IC94.9 (A7), ICR1.9 (R8)
Other:
- moved on the sheet: B16, IC10, IC11, IC12, IC13, IC14A, IC14B, IC15A, IC15B, IC15C, IC15D, IC18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

Commit message: wip video fairland
Parts:
- added IC30, IC6: 74LS86, symbol 74xx:74LS86
- added IC50, IC51: 74LS669, symbol 74xx_IEEE:74LS669
- added IC53: 74LS32, symbol jt74:74LS32
- added IC61: 74LS298, symbol jt74:74LS298
Connections:
- net ~{OE0} is gone; now on net ~{CHA3}: IC32.20 (~{CE}), IC32.22 (~{OE}), IC8.20 (~{CE}), IC8.22 (~{OE})
- net ~{OE1} is gone; now on net ~{CHA2}: IC33.20 (~{CE}), IC33.22 (~{OE}), IC9.20 (~{CE}), IC9.22 (~{OE})
- net ~{OE2} is gone; now on net ~{CHA1}: IC10.20 (~{CE}), IC10.22 (~{OE}), IC34.20 (~{CE}), IC34.22 (~{OE})
- net ~{OE3} is gone; now on net ~{CHA0}: IC11.20 (~{CE}), IC11.22 (~{OE}), IC35.20 (~{CE}), IC35.22 (~{OE})
- net CA10: now also IC21.13 (Qc)
- net CA11: now also IC21.12 (Qd)
- net CA4: now also IC7.15 (Qa)
- net CA5: now also IC7.14 (Qb)
- net CA6: now also IC7.13 (Qc)
- net CA7: now also IC7.12 (Qd)
- net CA8: now also IC21.15 (Qa)
- net CA9: now also IC21.14 (Qb)
- net FLIP7: no longer IC38.5
- net H1: now also IC70.13 (A2)
- net SUMD3': now also IC30.2
- net VCC: now also IC14.4 (~{S}), IC53.14 (VCC), IC61.16 (VCC)
- net VSS: now also IC20.1 (E), IC53.7 (VSS), IC61.8 (VSS)
- net at IC20.2 (A0): now also IC61.15 (Qa)
- net at IC20.3 (A1): now also IC61.14 (Qb)
- net ~{CHA0}: now reaches IC20.4 (O0)
- net ~{CHA1}: now reaches IC20.5 (O1)
- net ~{CHA2}: now reaches IC20.6 (O2)
- net ~{CHA3}: now reaches IC20.7 (O3)
- net SMX1: now reaches IC7.1 (I1b)
- net SMX1: now also IC30.8
- net SMX0: now reaches IC7.2 (I1a)
- net SMX0: now also IC30.3
- net ARAMDB0: now reaches IC7.5 (I1c)
- net ARAMDB0: now also IC45.18 (B0), IC62.2 (I1a), IC51.3 (P0)
- net ARAMDB1: now reaches IC7.6 (I1d)
- net ARAMDB1: now also IC45.17 (B1), IC62.1 (I1b), IC51.4 (P1)
- net ~{OUT0}: now reaches IC70.1 (0)
- net ~{OUT8}: now reaches IC70.10 (8)
- net ~{OUT9}: now reaches IC70.11 (9)
- net ~{OUT1}: now reaches IC70.2 (1)
- net ~{OUT2}: now reaches IC70.3 (2)
- net ~{OUT3}: now reaches IC70.4 (3)
- net ~{OUT4}: now reaches IC70.5 (4)
- net ~{OUT5}: now reaches IC70.6 (5)
- net ~{RST'}: now reaches IC70.7 (6)
- net ~{RST'}: now also IC14.1 (~{R}), IC53.10
- net ~{OUT7}: now reaches IC70.9 (7)
- net ARAMDB3: now reaches IC21.1 (I1b)
- net ARAMDB3: now also IC45.15 (B3), IC62.6 (I1d), IC51.6 (P3)
- net ARAMDB2: now reaches IC21.2 (I1a)
- net ARAMDB2: now also IC45.16 (B2), IC62.5 (I1c), IC51.5 (P2)
- net ARAMDB4: now reaches IC21.5 (I1c)
- net ARAMDB4: now also IC45.14 (B4)
- net ARAMDB5: now reaches IC21.6 (I1d)
- net ARAMDB5: now also IC45.13 (B5)
- net ARAMDB7: now reaches IC45.11 (B7)
- net ARAMDB7: now also IC61.6 (I1d)
- net ARAMDB6: now reaches IC45.12 (B6)
- net ARAMDB6: now also IC61.5 (I1c)
- net MUXd: now reaches IC47.3 (D0), IC62.12 (Qd)
- net MUXc: now reaches IC47.4 (D1), IC62.13 (Qc)
- net MUXb: now reaches IC47.7 (D2), IC62.14 (Qb)
- net MUXa: now reaches IC47.8 (D3), IC62.15 (Qa)
- net FFP5: now reaches IC46.15 (Q5)
- net FFP5: now also IC61.4 (I0b)
- net FFP1: now reaches IC46.5 (Q1)
- net FFP1: now also IC61.3 (I0a)
- net VF2: now reaches IC54.2 (Q0)
- net VF0: now reaches IC54.5 (Q1)
- net CLK' renamed CLK6M
- net CpFF renamed CPFF
- net MABD0 renamed MRAMD0
- net MABD1 renamed MRAMD1
- net MABD2 renamed MRAMD2
- net MABD3 renamed MRAMD3
- net MABD4 renamed MRAMD4
- net MABD5 renamed MRAMD5
- net MABD6 renamed MRAMD6
- net MABD7 renamed MRAMD7
- new net: IC30.9, IC61.13 (Qc)
- new net: IC30.1, IC6.5, IC61.12 (Qd)
- new net FLIARAMDB7: IC38.5
- new net P0: IC50.3 (P0), IC61.2 (I1a)
- new net P1: IC50.4 (P1), IC61.1 (I1b)
- new net P2: IC50.5 (P2)
- new net P3: IC50.6 (P3)
Other:
- note added: "1.54MHz"
- note added: "3.08MHz"
- note added: "4-bit binary counter synchronous"
- note added: "6.144MHz"
- note added: "6.25MHz"
- note added: "766KHz"
- note added: "769KHz"
- note added: "VERTICAL?"
- moved on the sheet: B16, IC10, IC11, IC12, IC13, IC14A, IC14B, IC15A, IC20A, IC20B, IC21, IC22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

Commit message: wip video fairyland
Parts:
- removed unit 5 of IC30
- removed unit 5 of IC53
- removed unit 5 of IC6
- added IC16, IC26: 74LS86, symbol jt74:74LS86
- added IC25: 74LS10, symbol jt74:74LS10
- added IC27: 74LS161, symbol jt74:74LS161
- added IC41: 74LS373, symbol jt74:74LS373
- added unit 5 of IC47
- added unit 2 of IC47
- added unit 4 of IC47
- added unit 6 of IC47
- added unit 3 of IC47
Connections:
- net FLIARAMDB7 is gone; now on net FLIP7: IC38.5
- net VF0 is gone; now on net SUMD0'': IC54.5 (Q1)
- net VF2 is gone; now on net SUMD2'': IC54.2 (Q0)
- net CA0: now also IC6.3
- net CA1: now also IC6.11
- net CA2: now also IC6.6
- net CA3: now also IC6.8
- net D3: now also IC15.9
- net D4: now also IC15.13, IC54.18 (D7)
- net D5: now also IC54.17 (D6)
- net D6: now also IC54.14 (D5)
- net D7: now also IC54.13 (D4)
- net H1: now also IC6.2
- net H2: now also IC30.10
- net MRAMD0: now also IC42.19 (O7), IC46.18 (D7), IC41.19 (O7)
- net MRAMD1: now also IC42.2 (O0), IC46.3 (D0), IC41.2 (O0)
- net MRAMD2: now also IC42.16 (O6), IC46.17 (D6), IC41.16 (O6)
- net MRAMD3: now also IC42.5 (O1), IC46.4 (D1), IC41.5 (O1)
- net MRAMD4: now also IC42.15 (O5), IC46.14 (D5), IC41.15 (O5)
- net MRAMD5: now also IC42.6 (O2), IC46.7 (D2), IC41.6 (O2)
- net MRAMD6: now also IC42.12 (O4), IC46.13 (D4), IC41.12 (O4)
- net MRAMD7: now also IC42.9 (O3), IC46.8 (D3), IC41.9 (O3)
- net SUMD7': now also IC55.16 (Q6)
- net VCC: now also IC54.1 (~{Mr}), IC16.14 (VCC), IC26.14 (VCC), IC27.1 (~{MR}), IC27.3 (D0), IC27.4 (D1), IC27.5 (D2), IC41.20 (VCC)
- net VSS: now also IC16.7 (VSS), IC26.7 (VSS), IC41.10 (VSS)
- net ~{OUT0}: no longer IC70.1 (0)
- net ~{OUT2}: no longer IC70.3 (2)
- net ~{OUT3}: no longer IC70.4 (3)
- net ~{OUT4}: no longer IC70.5 (4)
- net ~{OUT5}: no longer IC70.6 (5)
- net ~{OUT7}: no longer IC70.9 (7)
- net ~{OUT8}: no longer IC70.10 (8)
- net ~{OUT9}: no longer IC70.11 (9)
- net at IC30.9, IC61.13 (Qc): now also IC47.9
- net FLIP6: now reaches IC15.10
- net FLIP6: now also IC15.12, IC46.16 (Q6)
- net at IC15.8: now also IC38.4
- net at IC5.9 (Q): now also IC26.9
- net MRAMD6': now reaches IC76.15 (A9)
- net MRAMD6': now also IC46.12 (Q4)
- net at IC38.6: now also IC61.9 (I0c)
- net SUMB4: now reaches IC57.11 (B4)
- net SUMB4: now also IC16.6, IC41.4 (D1)
- net SUMB3: now reaches IC57.15 (B3)
- net SUMB3: now also IC16.8, IC41.17 (D6)
- net SUMB2: now reaches IC57.2 (B2)
- net SUMB2: now also IC16.3, IC41.3 (D0)
- net SUMB1: now reaches IC57.6 (B1)
- net SUMB1: now also IC26.8, IC41.18 (D7)
- net at IC30.1, IC6.5, IC61.12 (Qd): now also IC6.10, IC6.12
- net at IC61.7 (I0d): now also IC15.11
- net OEUK0: now reaches IC37.11, IC48.1 (~{OE}), IC95.17 (D6), IC96.11
- net at IC6.1: now also IC47.8
- net MRAMD5': now reaches IC82.17 (I3b)
- net MRAMD5': now also IC46.6 (Q2)
- net SUMD2'': now reaches IC6.9
- net SUMD0'': now reaches IC6.13
- net D6': now reaches IC31.3 (I0a), IC54.15 (Q5)
- net D7': now reaches IC31.4 (I0b), IC54.12 (Q4)
- net at IC46.2 (Q0): now also IC26.1, IC26.10, IC26.13, IC26.4
- net MRAMD7': now reaches IC46.9 (Q3)
- net SUMD1': now reaches IC55.9 (Q3)
- net SUMD1': now also IC54.8 (D3)
- net at IC54.7 (D2): now also IC25.12
- net SUMD1'': now reaches IC54.9 (Q3)
- net SUMD1'': now also IC6.4
- new net: IC25.4, IC26.12, IC27.13 (Q1)
- new net: IC27.10 (CET), IC27.7 (CEP)
- new net: IC26.5, IC27.12 (Q2)
- new net: IC26.2, IC27.14 (Q0)
- new net: IC26.3, IC41.7 (D2)
- new net: IC26.11, IC41.13 (D4)
- new net: IC16.11, IC41.14 (D5)
- new net: IC26.6, IC41.8 (D3)
- no-connect marks 9 -> 10
Other:
- note removed: "obj_lut_buf, COLMIX?"
- moved on the sheet: B16, IC10, IC11, IC12, IC13, IC14A, IC14B, IC15A, IC15B, IC15C, IC15D, IC18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

Commit message: sram video fairyland
Connections:
- net SRAD3: now reaches IC76.11 (D3)
- net SRAD3: now also IC91.14 (B4)
- net SRAD2: now reaches IC76.12 (D2)
- net SRAD2: now also IC91.13 (B5)
- net SRAD1: now reaches IC76.13 (D1)
- net SRAD1: now also IC91.12 (B6)
- net SRAD0: now reaches IC76.14 (D0)
- net SRAD0: now also IC91.11 (B7)
- net SRAD6: now reaches IC91.17 (B1), IC93.13 (D4)
- net SRAD6: now also IC77.12 (D2)
- net SRAD7: now reaches IC91.18 (B0), IC93.14 (D5)
- net SRAD7: now also IC77.11 (D3)
- net SRAD5: now reaches IC77.13 (D1)
- net SRAD5: now also IC91.16 (B2)
- net SRAD4: now reaches IC77.14 (D0)
- net SRAD4: now also IC91.15 (B3)
- net SRAD11: now reaches IC78.11 (D3)
- net SRAD11: now also IC94.14 (B4)
- net SRAD10: now reaches IC78.12 (D2)
- net SRAD10: now also IC94.13 (B5)
- net SRAD9: now reaches IC78.13 (D1)
- net SRAD9: now also IC94.12 (B6)
- net SRAD8: now reaches IC78.14 (D0)
- net SRAD8: now also IC94.11 (B7)
Other:
- moved on the sheet: B16, IC10, IC11, IC12, IC13, IC14A, IC14B, IC15A, IC15B, IC15C, IC15D, IC16A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

Commit message: wip fairyland video
Parts:
- added IC17: 74LS161, symbol jt74:74LS161
Connections:
- net VCC: now also IC17.1 (~{MR}), IC17.5 (D2), IC17.6 (D3)
- net VSS: now also IC17.3 (D0), IC17.4 (D1)
- net at IC5.11 (C): now also IC27.2 (CP), IC17.2 (CP)
- net QQ: now reaches IC26.9, IC5.9 (Q)
- net QQ: now also IC17.10 (CET), IC17.7 (CEP)
- net at IC16.10: now also IC16.1, IC16.13, IC16.4, IC26.1, IC26.10, IC26.13, IC26.4, IC46.2 (Q0)
- net at IC16.9: now also IC17.11 (Q3)
- net at IC16.2: now also IC17.14 (Q0)
- net X: now reaches IC16.11, IC41.14 (D5)
- net at IC16.12: now also IC17.13 (Q1)
- net at IC16.5: now also IC17.12 (Q2)
Other:
- moved on the sheet: IC16A, IC16B, IC16C, IC16D, IC26E, IC5B

Commit message: wip colmix faryland
Parts:
- added BR17: 10KΩ, symbol Device:R_US
- added BR20: 100KΩ, symbol Device:R_US
- added BR21: 47KΩ, symbol Device:R_US
- added BR22: 33KΩ, symbol Device:R_US
- added IC44: 74LS374, symbol jt74:74LS374
- added Q9: Q_NPN_ECB, symbol Device:Q_NPN_ECB
Connections:
- net RAMD0: now also IC44.3 (D0)
- net RAMD1: now also IC44.18 (D7)
- net RAMD2: now also IC44.4 (D1)
- net RAMD3: now also IC44.17 (D6)
- net RAMD4: now also IC44.7 (D2)
- net RAMD5: now also IC44.14 (D5)
- net RAMD6: now also IC44.8 (D3)
- net RAMD7: now also IC44.13 (D4)
- net VCC: now also Q9.2 (C)
- net at IC93.10 (Q3): now also BR17.1
- net at IC93.2 (Q0): now also BR20.1
- net at IC93.5 (Q1): now also BR21.1
- net at IC93.7 (Q2): now also BR22.1
- net at IC43.13 (D4): now also IC44.12 (O4)
- net at IC43.14 (D5): now also IC44.15 (O5)
- net at IC43.17 (D6): now also IC44.16 (O6)
- net at IC43.18 (D7): now also IC44.19 (O7)
- net at IC43.3 (D0): now also IC44.2 (O0)
- net at IC43.4 (D1): now also IC44.5 (O1)
- net at IC43.7 (D2): now also IC44.6 (O2)
- net at IC43.8 (D3): now also IC44.9 (O3)
Other:
- note added: "COLMIX?"
- note added: "OBJECTS?"
- note removed: "766KHz"
- note removed: "COLMIX SCROLL?"
- moved on the sheet: IC15B, IC16E, IC1B, IC24B, IC25C, IC26E, IC30B, IC30D, IC37B, IC37C, IC38C, IC38D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

Commit message: sch: changed copyright notice
Other:
- company: Esperanza Triana -> JOTEGO
Changed lines of the file:
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@@
     (date "2023-10-02")
     (rev "José Tejada G.")
-    (company "Esperanza Triana")
+    (company "JOTEGO")
     (comment 1 "www.patreon.com/jotego")
     (comment 2 "JOTEGO")
