File: cores/tmnt/sch/mia/io.kicad_sch (KiCad schematic)
At the start: 25 parts, among them SW1 SW3, SW1 SW_DIP_x08, SW2 SW_DIP_x08, U1 051550, U2 68000D, U3 74LS04

Commit message: page 4 of schematics m.i.a. #333, done!
Parts:
- removed RN7: R_Network08_US, Resistor_THT:R_Array_SIP9, symbol Device:R_Network08_US
- removed U2: 68000D, symbol CPU_NXP_68000:68000D
- added R1, R23: 470Ω, symbol Device:R_US
- added R2, R25: 100Ω, symbol Device:R_US
- added RN4: RA 2.2Kx 8, Resistor_THT:R_Array_SIP9, symbol Device:R_Network08_US
- RN2: renamed from RN8; value R_Network04_US -> RA 2.2Kx 4
- RN3: renamed from RN6; value R_Network08_US -> RA 2.2Kx 8
- renumbered U3 to F15
Connections:
- net AB1: now also A26.1 (S), B26.1 (S)
- net D0: now also A26.4 (Za), D29.12 (O3a)
- net D1: now also A26.7 (Zb), D29.14 (O2a)
- net D2: now also A26.12 (Zc), D29.16 (O1a)
- net D3: now also A26.9 (Zd), D29.18 (O0a)
- net D4: now also B26.4 (Za)
- net D5: now also B26.7 (Zb)
- net D6: now also B26.12 (Zc)
- net D7: now also B26.9 (Zd)
- net VCC: now also RN2.1 (common), RN3.1 (common), R1.1, R23.1, RN4.1 (common)
- net VSS: now also SW1.10, SW1.11, SW1.12, SW1.13, SW1.14, SW1.15, SW1.16, SW1.5, SW1.6, SW1.7, SW1.8, SW1.9, SW2.10, SW2.11, SW2.12, SW2.13, SW2.14, SW2.15, SW2.16, SW2.9
- net at B26.10 (I1d): now also SW2.8, RN4.9 (R8)
- net at B26.11 (I0d): now also RN3.9 (R8), SW1.8
- net at B26.13 (I1c): now also SW2.7, RN4.8 (R7)
- net at B26.14 (I0c): now also RN3.8 (R7), SW1.7
- net DIP: now reaches B26.15 (OE)
- net DIP: now also A26.15 (OE)
- net at B26.2 (I0a): now also RN3.6 (R5), SW1.5
- net at B26.3 (I1a): now also SW2.5, RN4.6 (R5)
- net at B26.5 (I0b): now also RN3.7 (R6), SW1.6
- net at B26.6 (I1b): now also SW2.6, RN4.7 (R6)
- net at RN3.2 (R1): now also A26.2 (I0a), SW1.1
- net at RN3.3 (R2): now also A26.5 (I0b), SW1.2
- net at RN3.4 (R3): now also A26.11 (I0d), SW1.3
- net at RN3.5 (R4): now also A26.14 (I0c), SW1.4
- net at RN2.2 (R1): now also D29.8 (I3a), SW1.1
- net at RN2.3 (R2): now also D29.6 (I2a), SW1.2
- net at RN2.4 (R3): now also D29.4 (I1a), SW1.3
- net at RN2.5 (R4): now also D29.2 (I0a), SW1.4
- net at SW2.1: now also A26.3 (I1a), RN4.2 (R1)
- net at SW2.2: now also A26.6 (I1b), RN4.3 (R2)
- net at SW2.3: now also A26.10 (I1d), RN4.4 (R3)
- net at SW2.4: now also A26.13 (I1c), RN4.5 (R4)
- net DIP3: now reaches D29.1 (OEa)
- net at D29.3 (O3b): now also R2.1
- net at D29.5 (O2b): now also R25.1
- net OIPL: now reaches D29.9 (O0b)
- new net SYNC: R23.2, R25.2
- new net ~{VSYNC}: R1.2, R2.2
Other:
- moved on the sheet: A26, B22, B26, C1, D29, FL1, JP1, RN2, RN3, SW1, SW2, U1
