File: cores/tmnt/sch/tmnt2/scroll.kicad_sch (KiCad schematic)
At the start: 7 parts, among them J13 051962

Commit message: extraccion finalizada, sch tmnt2 done!
Changed lines of the file:
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@@
     (effects (font (size 1.27 1.27)) (justify left))
   )
-  (hierarchical_label "MAIN_A[16..0]" (shape input) (at 34.29 198.12 180) (fields_autoplaced)
+  (hierarchical_label "MAIN_A[15..1]" (shape input) (at 34.29 198.12 180) (fields_autoplaced)
     (effects (font (size 1.27 1.27)) (justify right))
   )
