File: cores/risle/sch/io.kicad_sch (KiCad schematic)
At the start: 98 parts, among them IC53 TC0030CMD, IC54 74LS04, IC73 PC050CM, IC74 74LS02, IC77 74LS244, IC78 74LS244, IC79 74LS244, IC80 74LS04, X2 OSC-12.000MHz

Commit message: minor sch update
Parts:
- gave numbers to parts that had none: 1
- renumbered C11 to C100, C128 to C101, C128 to C102, C128 to C104, C11 to C84, C11 to C95, C11 to C97, C11 to C98, JP1 to JP2, L21 to L10, L21 to L11, L21 to L12, L41 to L13, L41 to L15, L21 to L20, L22 to L21, L23 to L22, L24 to L23, L25 to L24, L26 to L25, L21 to L7, L21 to L8, L21 to L9
