File: cores/risle/sch/tile_layers.kicad_sch (KiCad schematic)
At the start: 11 parts, among them IC14 74LS139, IC2 MN234000

Commit message: minor sch update
Parts:
- gave numbers to parts that had none: 9
