File: cores/twin16/sch/darkadv/scpu.kicad_sch (KiCad schematic)
At the start: 30 parts, among them K1 74LS32, M10 74LS245, M3.4 74LS02, M4 74LS21, M8 74LS138, M9 74LS245

Commit message: darkadv/twin16 finished cleaning up schematics and remaining issues
Parts:
- removed M4: 74LS21, symbol jt74:74LS21
- removed N10, N8, RR10, RRR8, S10, S8: 27512, Package_DIP:DIP-28_W15.24mm, symbol Memory_EPROM:27512
- removed UU10, UU8: 6264SL, symbol fujitsu:6264SL
- added AP_R10, A_N10, A_N8, A_R8, A_S10, A_S8: 27C512, symbol jt_rom:27C512
- added A_G5: 74LS74, symbol jt74:74LS74
- added A_M4: 74LS21, symbol 74xx:74LS21
- added A_U10, A_U8: 6264SL, symbol jt_ram:SRAM8K8B
- renumbered F6 to A_F6, F7 to A_F7, G6 to A_G6, H4 to A_H4, H5 to A_H5, H6 to A_H6, H7 to A_H7, H8 to A_H8, JJ1 to A_J1, JJ8 to A_J8, K1 to A_K1, L10 to A_L10, L9 to A_L9, M10 to A_M10, M3.4 to A_M3.4, M8 to A_M8, M9 to A_M9, RA7 to A_RA7, S7 to A_S7, TT7 to A_T7, V10 to A_V10
Connections:
- net GND: now also AP_R10.14 (GND), AP_R10.20 (~{CE}), A_N10.14 (GND), A_N10.20 (~{CE}), A_N8.14 (GND), A_N8.20 (~{CE}), A_R8.14 (GND), A_R8.20 (~{CE}), A_S10.14 (GND), A_S10.20 (~{CE}), A_S8.14 (GND), A_S8.20 (~{CE}), A_U10.14 (GND), A_U8.14 (GND)
- net SA15: now also AP_R10.27 (A14), A_N10.27 (A14), A_N8.27 (A14), A_R8.27 (A14), A_S10.27 (A14), A_S8.27 (A14)
- net SA16: now also AP_R10.1 (A15), A_N10.1 (A15), A_N8.1 (A15), A_R8.1 (A15), A_S10.1 (A15), A_S8.1 (A15)
- net SAB1: now also AP_R10.10 (A0), A_N10.10 (A0), A_N8.10 (A0), A_R8.10 (A0), A_S10.10 (A0), A_S8.10 (A0), A_U10.10 (A0), A_U8.2 (A12)
- net SAB10: now also AP_R10.24 (A9), A_N10.24 (A9), A_N8.24 (A9), A_R8.24 (A9), A_S10.24 (A9), A_S8.24 (A9), A_U10.24 (A9), A_U8.7 (A3)
- net SAB11: now also AP_R10.21 (A10), A_N10.21 (A10), A_N8.21 (A10), A_R8.21 (A10), A_S10.21 (A10), A_S8.21 (A10), A_U10.21 (A10), A_U8.8 (A2)
- net SAB12: now also AP_R10.23 (A11), A_N10.23 (A11), A_N8.23 (A11), A_R8.23 (A11), A_S10.23 (A11), A_S8.23 (A11), A_U10.23 (A11), A_U8.9 (A1)
- net SAB13: now also AP_R10.2 (A12), A_N10.2 (A12), A_N8.2 (A12), A_R8.2 (A12), A_S10.2 (A12), A_S8.2 (A12), A_U10.2 (A12), A_U8.10 (A0)
- net SAB14: now also AP_R10.26 (A13), A_N10.26 (A13), A_N8.26 (A13), A_R8.26 (A13), A_S10.26 (A13), A_S8.26 (A13)
- net SAB2: now also AP_R10.9 (A1), A_N10.9 (A1), A_N8.9 (A1), A_R8.9 (A1), A_S10.9 (A1), A_S8.9 (A1), A_U10.9 (A1), A_U8.23 (A11)
- net SAB3: now also AP_R10.8 (A2), A_N10.8 (A2), A_N8.8 (A2), A_R8.8 (A2), A_S10.8 (A2), A_S8.8 (A2), A_U10.8 (A2), A_U8.21 (A10)
- net SAB4: now also AP_R10.7 (A3), A_N10.7 (A3), A_N8.7 (A3), A_R8.7 (A3), A_S10.7 (A3), A_S8.7 (A3), A_U10.7 (A3), A_U8.24 (A9)
- net SAB5: now also AP_R10.6 (A4), A_N10.6 (A4), A_N8.6 (A4), A_R8.6 (A4), A_S10.6 (A4), A_S8.6 (A4), A_U10.6 (A4), A_U8.25 (A8)
- net SAB6: now also AP_R10.5 (A5), A_N10.5 (A5), A_N8.5 (A5), A_R8.5 (A5), A_S10.5 (A5), A_S8.5 (A5), A_U10.5 (A5), A_U8.3 (A7)
- net SAB7: now also AP_R10.4 (A6), A_N10.4 (A6), A_N8.4 (A6), A_R8.4 (A6), A_S10.4 (A6), A_S8.4 (A6), A_U10.4 (A6), A_U8.4 (A6)
- net SAB8: now also AP_R10.3 (A7), A_N10.3 (A7), A_N8.3 (A7), A_R8.3 (A7), A_S10.3 (A7), A_S8.3 (A7), A_U10.3 (A7), A_U8.5 (A5)
- net SAB9: now also AP_R10.25 (A8), A_N10.25 (A8), A_N8.25 (A8), A_R8.25 (A8), A_S10.25 (A8), A_S8.25 (A8), A_U10.25 (A8), A_U8.6 (A4)
- net SDB0: now also A_N8.11 (D0), A_R8.11 (D0), A_S8.11 (D0), A_U8.11 (D0)
- net SDB1: now also A_N8.12 (D1), A_R8.12 (D1), A_S8.12 (D1), A_U8.12 (D1)
- net SDB10: now also AP_R10.13 (D2), A_N10.13 (D2), A_S10.13 (D2), A_U10.13 (D2)
- net SDB11: now also AP_R10.15 (D3), A_N10.15 (D3), A_S10.15 (D3), A_U10.15 (D3)
- net SDB12: now also AP_R10.16 (D4), A_N10.16 (D4), A_S10.16 (D4), A_U10.16 (D4)
- net SDB13: now also AP_R10.17 (D5), A_N10.17 (D5), A_S10.17 (D5), A_U10.17 (D5)
- net SDB14: now also AP_R10.18 (D6), A_N10.18 (D6), A_S10.18 (D6), A_U10.18 (D6)
- net SDB15: now also AP_R10.19 (D7), A_N10.19 (D7), A_S10.19 (D7), A_U10.19 (D7)
- net SDB2: now also A_G5.2 (D), A_N8.13 (D2), A_R8.13 (D2), A_S8.13 (D2), A_U8.13 (D2)
- net SDB3: now also A_N8.15 (D3), A_R8.15 (D3), A_S8.15 (D3), A_U8.15 (D3)
- net SDB4: now also A_N8.16 (D4), A_R8.16 (D4), A_S8.16 (D4), A_U8.16 (D4)
- net SDB5: now also A_N8.17 (D5), A_R8.17 (D5), A_S8.17 (D5), A_U8.17 (D5)
- net SDB6: now also A_N8.18 (D6), A_R8.18 (D6), A_S8.18 (D6), A_U8.18 (D6)
- net SDB7: now also A_N8.19 (D7), A_R8.19 (D7), A_S8.19 (D7), A_U8.19 (D7)
- net SDB8: now also AP_R10.11 (D0), A_N10.11 (D0), A_S10.11 (D0), A_U10.11 (D0)
- net SDB9: now also AP_R10.12 (D1), A_N10.12 (D1), A_S10.12 (D1), A_U10.12 (D1)
- net VCC: now also A_L9.16 (VCC), AP_R10.28 (VCC), A_G5.1 (~{R}), A_G5.4 (~{S}), A_M4.1, A_N10.28 (VCC), A_N8.28 (VCC), A_R8.28 (VCC), A_S10.28 (VCC), A_S8.28 (VCC), A_U10.26 (CS2), A_U10.28 (VCC), A_U8.26 (CS2), A_U8.28 (VCC)
- net VSS: now also A_L9.8 (VSS)
- net ~{OCHAROMCS}: now also A_M4.6
- net ~{SLWR}: now also A_U8.27 (~{WR})
- net ~{SREAD}: now also A_U10.22 (~{OE}), A_U8.22 (~{OE})
- net ~{SSYSFLAG}: now also A_G5.3 (C)
- net ~{SUWR}: now also A_U10.27 (~{WR})
- net ~{SWORKCS}: now also A_U10.20 (~{CS1}), A_U8.20 (~{CS1})
- net at A_M8.11 (O4): now also AP_R10.22 (~{OE}), A_R8.22 (~{OE})
- net at A_M8.14 (O1): now also A_S10.22 (~{OE}), A_S8.22 (~{OE})
- net at A_M8.15 (O0): now also A_N10.22 (~{OE}), A_N8.22 (~{OE})
- net at A_T7.9 (O6): now also A_M4.2
- net at A_T7.10 (O5): now also A_M4.4
- net at A_T7.11 (O4): now also A_M4.5
- new net CHAPAGE: A_G5.5 (Q)
- no-connect marks 16 -> 17
Other:
- note added: "Only used on PWB(A)302190B Goes to CN2:24. On PWB(A)302190A CN2:24 is connected to GND."
- title: Dark Adventure / Gradius 2 -> Twin 16
- moved on the sheet: A_H7D

Commit message: minor
Other:
- note added: "Only used on PWB(A)302190B Goes to CN2:A23. On PWB(A)302190A CN2:A23 is connected to GND."
- note removed: "Only used on PWB(A)302190B Goes to CN2:24. On PWB(A)302190A CN2:24 is connected to GND."
Changed lines of the file:
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@@
     (effects (font (size 1.27 1.27)) (justify left bottom))
   )
-  (text "Only used on PWB(A)302190B\nGoes to CN2:24.\nOn PWB(A)302190A CN2:24 is connected to GND."
+  (text "Only used on PWB(A)302190B\nGoes to CN2:A23.\nOn PWB(A)302190A CN2:A23 is connected to GND."
     (at 67.31 53.34 0)
     (effects (font (size 1.27 1.27)) (justify left bottom))
