File: cores/wwfss/sch/wwfsstar.kicad_sch (KiCad schematic)
At the start: 0 parts

Commit message: schematic work
Other:
- sheet bottom ports: added D~{O}BJHP[0..7], ER[0..7], MA[1..11], MA[1..12], MD[0..7], OBJCOL[0..3], OBJPXL[0..6], TEL[0..7]; removed none
- sheet top ports: added MA[1..16], MD[0..15], OBJPXL[0..6], SCRPXL1[0..6]; removed none
- note removed: "THIS IS THE LATEST VERSION"
