File: cores/twin16/sch/007785/counters.kicad_sch (KiCad schematic)
At the start: 79 parts, among them J3 ENR, J30 2AD, J34 DFR, J8 ENR, K3 D1A, K32 2OR, K41 DFR, K7 2ND, M30 DFR, M40 JKFR, P14 ENR, P39 DFR, Q24 DFR, Q3 3ND, T11 3AD, T15 2ND, T18 4AD, T23 EXR, T3 2AD, T31 2AD, T35 2AD, T39 DFR, T60 INV, T7 D1A, U16 ENR, U24 ENR, U3 3ND, U30 3ND, U39 DFR, U7 3ND

Commit message: Corrected tri-state buffers to output enable active high
Connections:
- net at F31.: now also D36.; no longer K32.
- new net: F31., K32.
- new net: F31., M40. (~{Q})
- new net: N3., W4.
- new net: V7., W4.
- new net: T35., U16.
- new net: S40. (~{Q}), T35.
- new net: N11., T15.
- new net: C35., N11.
- new net: N52., N57.
- new net: O3., U3.
- new net: W28., W9.
- new net: S11., U16.
- new net: C27., D15.
- new net: C27., G35. (~{Q})
- new net: R22., W14.
- new net: E34., E38. (~{Q})
- new net: E34., J3.
- new net: N7., P14.
- new net: T11., U7.
- new net: G27., G7.
- new net: U3., V7.
- new net: Q24. (~{Q}), T31.
- new net: U24., W42.
- new net: W42., W47. (~{Q})
- new net: T18., V34.
- new net: G10., L3.
- new net: V15., W37.
- new net: V25., W28.
- new net: V25., W19.
- new net: V25., V34.
- new net: U30., V25.
- new net: J30., M30. (~{Q})
- new net: B27., J34. (~{Q})
- new net: B27., G10.
- new net: T23., T31.
- new net: C31., R22.
- new net: T39. (~{Q}), W37.
- new net: D40., N52.
- new net: C35., L34. (~{Q})
- new net: D32., K41. (~{Q})
- new net: C31., P39. (~{Q})
- new net: D44., G27.
- new net: D44., F34. (~{Q})
- new net: U7., V7.
- new net: T3., U30.
- new net: U24., V11.
- new net: R28., R44.
- new net: R44., T60.
- new net: S7., V7.
- new net: J3., K7.
- new net: D32., P14.
- new net: S20., V39.
- new net: J8., Q3.
- new net: J30., J8.
- new net: U39. (~{Q}), V39.
Changed lines of the file:
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@@
   (paper "A3")
   (title_block
-    (date "2023-11-18")
+    (date "2023-12-22")
   )
   (bus_alias "HCOUNT" (members "H8" "H16" "H32" "H64"))

Commit message: updated references to jtkicad libraries
Connections:
- net at F31.: now also D36.; no longer K32.
- new net: F31., K32.
- new net: F31., M40. (~{Q})
- new net: N3., W4.
- new net: V7., W4.
- new net: T35., U16.
- new net: S40. (~{Q}), T35.
- new net: N11., T15.
- new net: C35., N11.
- new net: N52., N57.
- new net: O3., U3.
- new net: W28., W9.
- new net: S11., U16.
- new net: C27., D15.
- new net: C27., G35. (~{Q})
- new net: R22., W14.
- new net: E34., E38. (~{Q})
- new net: E34., J3.
- new net: N7., P14.
- new net: T11., U7.
- new net: G27., G7.
- new net: U3., V7.
- new net: Q24. (~{Q}), T31.
- new net: U24., W42.
- new net: W42., W47. (~{Q})
- new net: T18., V34.
- new net: G10., L3.
- new net: V15., W37.
- new net: V25., W28.
- new net: V25., W19.
- new net: V25., V34.
- new net: U30., V25.
- new net: J30., M30. (~{Q})
- new net: B27., J34. (~{Q})
- new net: B27., G10.
- new net: T23., T31.
- new net: C31., R22.
- new net: T39. (~{Q}), W37.
- new net: D40., N52.
- new net: C35., L34. (~{Q})
- new net: D32., K41. (~{Q})
- new net: C31., P39. (~{Q})
- new net: D44., G27.
- new net: D44., F34. (~{Q})
- new net: U7., V7.
- new net: T3., U30.
- new net: U24., V11.
- new net: R28., R44.
- new net: R44., T60.
- new net: S7., V7.
- new net: J3., K7.
- new net: D32., P14.
- new net: S20., V39.
- new net: J8., Q3.
- new net: J30., J8.
- new net: U39. (~{Q}), V39.

Commit message: changed symbol FDN to active low symbol. Updated to correct name for OKI Gate Arrays.
Parts:
- B27, C27, C31, C35, D32, D40, D44, E34, J30, O3, T3, T31, T35, V39, W37, W42: symbol oki-msm70v000:2AD -> ga_oki_msm70v0000:2AD
- D15, S20, T23, V15: symbol oki-msm70v000:EXR -> ga_oki_msm70v0000:EXR
- D36, K32: symbol oki-msm70v000:2OR -> ga_oki_msm70v0000:2OR
- E38, F34, G35, J34, K41, L34, M30, P39, Q24, S40, T39, U39, W47: symbol oki-msm70v000:DFR -> ga_oki_msm70v0000:DFR
- F31: symbol oki-msm70v000:2NR -> ga_oki_msm70v0000:2NR
- G10, G27, J3, J8, N11, P14, R22, U16, U24: symbol oki-msm70v000:ENR -> ga_oki_msm70v0000:ENR
- G7, K7, S11, T15: symbol oki-msm70v000:2ND -> ga_oki_msm70v0000:2ND
- K3, R28, S3, T7: symbol oki-msm70v000:D1A -> ga_oki_msm70v0000:D1A
- L3, Q3, S7, U3, U30, U7, V34, W14, W19, W28, W4: symbol oki-msm70v000:3ND -> ga_oki_msm70v0000:3ND
- M40: symbol oki-msm70v000:JKFR -> ga_oki_msm70v0000:JKFR
- N16, S14: symbol oki-msm70v000:5AD -> ga_oki_msm70v0000:5AD
- N3, T11, W9: symbol oki-msm70v000:3AD -> ga_oki_msm70v0000:3AD
- N52, R44: symbol oki-msm70v000:220 -> ga_oki_msm70v0000:220
- N57, T60: symbol oki-msm70v000:INV -> ga_oki_msm70v0000:INV
- N7, V11, V25, V7: symbol oki-msm70v000:4ND -> ga_oki_msm70v0000:4ND
- T18: symbol oki-msm70v000:4AD -> ga_oki_msm70v0000:4AD
Connections:
- net at F31.: now also D36.; no longer K32.
- new net: F31., K32.
- new net: F31., M40. (~{Q})
- new net: N3., W4.
- new net: V7., W4.
- new net: T35., U16.
- new net: S40. (~{Q}), T35.
- new net: N11., T15.
- new net: C35., N11.
- new net: N52., N57.
- new net: O3., U3.
- new net: W28., W9.
- new net: S11., U16.
- new net: C27., D15.
- new net: C27., G35. (~{Q})
- new net: R22., W14.
- new net: E34., E38. (~{Q})
- new net: E34., J3.
- new net: N7., P14.
- new net: T11., U7.
- new net: G27., G7.
- new net: U3., V7.
- new net: Q24. (~{Q}), T31.
- new net: U24., W42.
- new net: W42., W47. (~{Q})
- new net: T18., V34.
- new net: G10., L3.
- new net: V15., W37.
- new net: V25., W28.
- new net: V25., W19.
- new net: V25., V34.
- new net: U30., V25.
- new net: J30., M30. (~{Q})
- new net: B27., J34. (~{Q})
- new net: B27., G10.
- new net: T23., T31.
- new net: C31., R22.
- new net: T39. (~{Q}), W37.
- new net: D40., N52.
- new net: C35., L34. (~{Q})
- new net: D32., K41. (~{Q})
- new net: C31., P39. (~{Q})
- new net: D44., G27.
- new net: D44., F34. (~{Q})
- new net: U7., V7.
- new net: T3., U30.
- new net: U24., V11.
- new net: R28., R44.
- new net: R44., T60.
- new net: S7., V7.
- new net: J3., K7.
- new net: D32., P14.
- new net: S20., V39.
- new net: J8., Q3.
- new net: J30., J8.
- new net: U39. (~{Q}), V39.

Commit message: 007785 - minor edits
Connections:
- net at F31.: now also D36.; no longer K32.
- new net: F31., K32.
- new net: F31., M40. (~{Q})
- new net: N3., W4.
- new net: V7., W4.
- new net: T35., U16.
- new net: S40. (~{Q}), T35.
- new net: N11., T15.
- new net: C35., N11.
- new net: N52., N57.
- new net: O3., U3.
- new net: W28., W9.
- new net: S11., U16.
- new net: C27., D15.
- new net: C27., G35. (~{Q})
- new net: R22., W14.
- new net: E34., E38. (~{Q})
- new net: E34., J3.
- new net: N7., P14.
- new net: T11., U7.
- new net: G27., G7.
- new net: U3., V7.
- new net: Q24. (~{Q}), T31.
- new net: U24., W42.
- new net: W42., W47. (~{Q})
- new net: T18., V34.
- new net: G10., L3.
- new net: V15., W37.
- new net: V25., W28.
- new net: V25., W19.
- new net: V25., V34.
- new net: U30., V25.
- new net: J30., M30. (~{Q})
- new net: B27., J34. (~{Q})
- new net: B27., G10.
- new net: T23., T31.
- new net: C31., R22.
- new net: T39. (~{Q}), W37.
- new net: D40., N52.
- new net: C35., L34. (~{Q})
- new net: D32., K41. (~{Q})
- new net: C31., P39. (~{Q})
- new net: D44., G27.
- new net: D44., F34. (~{Q})
- new net: U7., V7.
- new net: T3., U30.
- new net: U24., V11.
- new net: R28., R44.
- new net: R44., T60.
- new net: S7., V7.
- new net: J3., K7.
- new net: D32., P14.
- new net: S20., V39.
- new net: J8., Q3.
- new net: J30., J8.
- new net: U39. (~{Q}), V39.
