File: cores/riders/sch/dbz/ROM2.kicad_sch (KiCad schematic)
At the start: 22 parts

Commit message: dbz sch
Connections:
- net 16JCLK renamed 15E9
- net MOROE3 renamed MOROE4
- net RAB0 renamed RB0
- net RAB1 renamed RB1
- net RAB10 renamed RB10
- net RAB11 renamed RB11
- net RAB12 renamed RB12
- net RAB13 renamed RB13
- net RAB14 renamed RB14
- net RAB15 renamed RB15
- net RAB16 renamed RB16
- net RAB17 renamed RB17
- net RAB18 renamed RB18
- net RAB19 renamed RB19
- net RAB2 renamed RB2
- net RAB3 renamed RB3
- net RAB4 renamed RB4
- net RAB5 renamed RB5
- net RAB6 renamed RB6
- net RAB7 renamed RB7
- net RAB8 renamed RB8
- net RAB9 renamed RB9
- net RAB_LOW renamed RB_LOW
- net XB0 renamed X0
- net XB1 renamed X1
- net XB2 renamed X2
- net XB3 renamed X3
- net XB4 renamed X4
- net XB5 renamed X5
- net XB6 renamed X6
- net XB7 renamed X7
- net XB8 renamed X8
- net XB9 renamed X9
- net YB0 renamed Y0
- net YB1 renamed Y1
- net YB2 renamed Y2
- net YB3 renamed Y3
- net YB4 renamed Y4
- net YB5 renamed Y5
- net YB6 renamed Y6
- net YB7 renamed Y7
- net YB8 renamed Y8
Other:
- note removed: "TO UNPOPULATED"
- moved on the sheet: 10HA, 15G, 17F, 19H, 22G, 22H, 23GA, 23GB, 23GD, 23H, 24H, 24J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

Commit message: minor
Changed lines of the file:
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@@
 	)
 	(bus_entry
-		(at 260.35 24.13)
-		(size 2.54 2.54)
-		(stroke
-			(width 0)
-			(type default)
-		)
-	)
-	(bus_entry
 		(at 83.82 109.22)
 		(size 2.54 2.54)
@@
 	)
 	(bus_entry
-		(at 260.35 81.28)
-		(size 2.54 2.54)
-		(stroke
-			(width 0)
-			(type default)
-		)
-	)
-	(bus_entry
 		(at 260.35 124.46)
 		(size 2.54 2.54)
@@
 	(bus
 		(pts
-			(xy 262.89 83.82) (xy 262.89 86.36)
+			(xy 262.89 41.91) (xy 262.89 86.36)
 		)
 		(stroke
@@
 	(wire
 		(pts
-			(xy 250.19 81.28) (xy 260.35 81.28)
+			(xy 250.19 81.28) (xy 259.08 81.28)
 		)
 		(stroke
@@
 		)
 	)
-	(bus
-		(pts
-			(xy 262.89 41.91) (xy 262.89 83.82)
-		)
-		(stroke
-			(width 0)
-			(type default)
-		)
-	)
 	(wire
 		(pts
@@
 	)
 	(label "RB_LOW"
-		(at 257.81 81.28 180)
+		(at 259.08 81.28 180)
 		(effects
 			(font
